Commit message: added excavator stuff for nav2

File: urdf_visualize/urdf/robot_wheel.xacro (robot description, xacro)
@@ -2,5 +2,5 @@
 <robot xmlns:xacro="http://www.ros.org/wiki/xacro" name="onshape">
     <!-- <link name="world"/> -->
-    <xacro:property name="mesh_root" value="package://urdf_visualize/meshes"/>
+    <xacro:property name="mesh_root" value="file://$(find urdf_visualize)/meshes"/>
     <xacro:property name="cabin_base_mesh" value="${mesh_root}/compact_excavator_cabin_body.stl"/>
     <xacro:property name="cabin_base_origin" value="0.1592 -0.2513 0.2814"/>
@@ -46,5 +46,5 @@
             <origin xyz="1.232595164407830946e-32 8.7258015952359883014e-17 -0.11999999999999998168" rpy="0 0 0" />
             <geometry>
-                <mesh filename="package://urdf_visualize/meshes/compact_excavator_frame_body.stl"/>
+                <mesh filename="file://$(find urdf_visualize)/meshes/compact_excavator_frame_body.stl"/>
             </geometry>
                 <material name="compact_excavator_frame_body_material">
@@ -55,5 +55,5 @@
             <origin xyz="1.232595164407830946e-32 8.7258015952359883014e-17 -0.11999999999999998168" rpy="0 0 0" />
             <geometry>
-            <mesh filename="package://urdf_visualize/meshes/compact_excavator_frame_body.stl"/>
+            <mesh filename="file://$(find urdf_visualize)/meshes/compact_excavator_frame_body.stl"/>
             </geometry>
         </collision>
@@ -90,5 +90,5 @@
             <origin xyz="0 -2.0816681711721685133e-17 -0.015000000000000124345" rpy="-4.71 0 0" />
             <geometry>
-            <mesh filename="package://urdf_visualize/meshes/compact_excavator_main_drive_wheel.stl"/>
+            <mesh filename="${mesh_root}/compact_excavator_main_drive_wheel.stl"/>
             </geometry>
             <material name="compact_excavator_main_drive_wheel_material">
@@ -99,5 +99,5 @@
             <origin xyz="0 -2.0816681711721685133e-17 -0.015000000000000124345" rpy="-4.71 0 0" />
             <geometry>
-            <mesh filename="package://urdf_visualize/meshes/compact_excavator_main_drive_wheel.stl"/>
+            <mesh filename="${mesh_root}/compact_excavator_main_drive_wheel.stl"/>
             </geometry>
         </collision>
@@ -112,5 +112,5 @@
             <origin xyz="-6.9388939039072283776e-18 0 -0.015000000000000013323" rpy="1.57 0 0" />
             <geometry>
-            <mesh filename="package://urdf_visualize/meshes/compact_excavator_main_drive_wheel.stl"/>
+            <mesh filename="${mesh_root}/compact_excavator_main_drive_wheel.stl"/>
             </geometry>
             <material name="compact_excavator_main_drive_wheel_material">
@@ -121,5 +121,5 @@
             <origin xyz="-6.9388939039072283776e-18 0 -0.015000000000000013323" rpy="1.57 0 0" />
             <geometry>
-            <mesh filename="package://urdf_visualize/meshes/compact_excavator_main_drive_wheel.stl"/>
+            <mesh filename="${mesh_root}/compact_excavator_main_drive_wheel.stl"/>
             </geometry>
         </collision>
@@ -134,5 +134,5 @@
             <origin xyz="1.1102230246251565404e-16 -1.1102230246251565404e-16 -0.032500000000000084377" rpy="0 1.570796326794896336 0" />
             <geometry>
-            <mesh filename="package://urdf_visualize/meshes/compact_excavator_front_wheel.stl"/>
+            <mesh filename="${mesh_root}/compact_excavator_front_wheel.stl"/>
             </geometry>
             <material name="compact_excavator_front_wheel_material">
@@ -143,5 +143,5 @@
             <origin xyz="1.1102230246251565404e-16 -1.1102230246251565404e-16 -0.032500000000000084377" rpy="0 1.570796326794896336 0" />
             <geometry>
-            <mesh filename="package://urdf_visualize/meshes/compact_excavator_front_wheel.stl"/>
+            <mesh filename="${mesh_root}/compact_excavator_front_wheel.stl"/>
             </geometry>
         </collision>
@@ -156,5 +156,5 @@
             <origin xyz="0 0 -0.032500000000000084377" rpy="-3.14 -1.570796326794896336 0" />
             <geometry>
-            <mesh filename="package://urdf_visualize/meshes/compact_excavator_front_wheel.stl"/>
+            <mesh filename="${mesh_root}/compact_excavator_front_wheel.stl"/>
             </geometry>
             <material name="compact_excavator_front_wheel_material">
@@ -165,5 +165,5 @@
             <origin xyz="0 0 -0.032500000000000084377" rpy="-3.14 -1.570796326794896336 0" />
             <geometry>
-            <mesh filename="package://urdf_visualize/meshes/compact_excavator_front_wheel.stl"/>
+            <mesh filename="${mesh_root}/compact_excavator_front_wheel.stl"/>
             </geometry>
         </collision>
@@ -178,5 +178,5 @@
             <origin xyz="-0.021564399534920564161 1.0799900599760599018 -0.25500000000000000444" rpy="-3.14 -1.57 0" />
             <geometry>
-            <mesh filename="package://urdf_visualize/meshes/push_blade_bucket.stl"/>
+            <mesh filename="${mesh_root}/push_blade_bucket.stl"/>
             </geometry>
             <material name="push_blade_bucket_material">
@@ -187,5 +187,5 @@
             <origin xyz="-0.021564399534920564161 1.0799900599760599018 -0.25500000000000000444" rpy="-3.14 -1.57 0" />
             <geometry>
-            <mesh filename="package://urdf_visualize/meshes/push_blade_bucket.stl"/>
+            <mesh filename="${mesh_root}/push_blade_bucket.stl"/>
             </geometry>
         </collision>
@@ -200,5 +200,5 @@
             <origin xyz="2.7755575615628913511e-17 0.074999999999999955591 -0.14999999999999996669" rpy="-3.14 -6.1629758220391547298e-33 -3.9110122218931175387e-17" />
             <geometry>
-            <mesh filename="package://urdf_visualize/meshes/part01_pin_1.stl"/>
+            <mesh filename="${mesh_root}/part01_pin_1.stl"/>
             </geometry>
             <material name="part01_pin_1_material">
@@ -209,5 +209,5 @@
             <origin xyz="2.7755575615628913511e-17 0.074999999999999955591 -0.14999999999999996669" rpy="-3.14 -6.1629758220391547298e-33 -3.9110122218931175387e-17" />
             <geometry>
-            <mesh filename="package://urdf_visualize/meshes/part01_pin_1.stl"/>
+            <mesh filename="${mesh_root}/part01_pin_1.stl"/>
             </geometry>
         </collision>
@@ -222,5 +222,5 @@
             <origin xyz="0 -1.1102230246251565404e-16 -0.079999999999999987788" rpy="-1.57 0 0" />
             <geometry>
-            <mesh filename="package://urdf_visualize/meshes/part02.stl"/>
+            <mesh filename="${mesh_root}/part02.stl"/>
             </geometry>
             <material name="part02_material">
@@ -231,5 +231,5 @@
             <origin xyz="0 -1.1102230246251565404e-16 -0.079999999999999987788" rpy="-1.57 0 0" />
             <geometry>
-            <mesh filename="package://urdf_visualize/meshes/part02.stl"/>
+            <mesh filename="${mesh_root}/part02.stl"/>
             </geometry>
         </collision>
@@ -244,5 +244,5 @@
             <origin xyz="0 -2.2204460492503130808e-16 -0.054999999999999882316" rpy="1.57 0 0" />
             <geometry>
-            <mesh filename="package://urdf_visualize/meshes/part03.stl"/>
+            <mesh filename="${mesh_root}/part03.stl"/>
             </geometry>
             <material name="part03_material">
@@ -253,5 +253,5 @@
             <origin xyz="0 -2.2204460492503130808e-16 -0.054999999999999882316" rpy="1.57 0 0" />
             <geometry>
-            <mesh filename="package://urdf_visualize/meshes/part03.stl"/>
+            <mesh filename="${mesh_root}/part03.stl"/>
             </geometry>
         </collision>
@@ -266,5 +266,5 @@
             <origin xyz="0.060000000000000053291 0.14000000000000012434 0.054999999999999993339" rpy="-3.14 -1.57 0" />
             <geometry>
-            <mesh filename="package://urdf_visualize/meshes/part04.stl"/>
+            <mesh filename="${mesh_root}/part04.stl"/>
             </geometry>
             <material name="part04_material">
@@ -275,5 +275,5 @@
             <origin xyz="0.060000000000000053291 0.14000000000000012434 0.054999999999999993339" rpy="-3.14 -1.57 0" />
             <geometry>
-            <mesh filename="package://urdf_visualize/meshes/part04.stl"/>
+            <mesh filename="${mesh_root}/part04.stl"/>
             </geometry>
         </collision>
@@ -281,5 +281,5 @@
             <origin xyz="0.078718096856630614955 0.97961106773940276327 0.054999999999992416067" rpy="-1.57 0 3" />
             <geometry>
-            <mesh filename="package://urdf_visualize/meshes/bucket.stl"/>
+            <mesh filename="${mesh_root}/bucket.stl"/>
             </geometry>
             <material name="bucket_material">
@@ -290,5 +290,5 @@
             <origin xyz="0.078718096856630614955 0.97961106773940276327 0.054999999999992416067" rpy="-1.57 0 3" />
             <geometry>
-            <mesh filename="package://urdf_visualize/meshes/bucket.stl"/>
+            <mesh filename="${mesh_root}/bucket.stl"/>
             </geometry>
         </collision>
@@ -296,5 +296,5 @@
             <origin xyz="0.16999999999999237943 0.30800000000000604672 0.054999999999999299449" rpy="-4.71 -1.57 0" />
             <geometry>
-            <mesh filename="package://urdf_visualize/meshes/bucket_mount.stl"/>
+            <mesh filename="${mesh_root}/bucket_mount.stl"/>
             </geometry>
             <material name="bucket_mount_material">
@@ -305,5 +305,5 @@
             <origin xyz="0.16999999999999237943 0.30800000000000604672 0.054999999999999299449" rpy="-4.71 -1.57 0" />
             <geometry>
-            <mesh filename="package://urdf_visualize/meshes/bucket_mount.stl"/>
+            <mesh filename="${mesh_root}/bucket_mount.stl"/>
             </geometry>
         </collision>
@@ -409,4 +409,13 @@
         </inertial>
     </link>
+    <xacro:macro name="gazebo_joints">
+        <!-- <gazebo>
+            <joint>
+                <stiffness>100000.0</stiffness>
+                <damping>5</damping>
+            </joint>
+        </gazebo>
+        <joint_properties damping="5" friction="0.9"/> -->
+    </xacro:macro>
     <joint name="left_spinning_wheel_joint" type="continuous">
         <origin xyz="0 0 -0.3" rpy="0 0 0"/>
@@ -415,5 +424,6 @@
         <axis xyz="0 0 1"/>
         <limit effort="1" velocity="20"/>
-        <joint_properties friction="0.0"/>
+        <!-- <joint_properties friction="0.0"/> -->
+        <xacro:gazebo_joints/>
     </joint>
     <joint name="left_passive_wheel_joint" type="continuous">
@@ -423,5 +433,6 @@
         <axis xyz="0 0 1"/>
         <limit effort="1" velocity="20"/>
-        <joint_properties friction="0.0"/>
+        <!-- <joint_properties friction="0.0"/> -->
+        <xacro:gazebo_joints/>
     </joint>
     <joint name="right_spinning_wheel_joint" type="continuous">
@@ -431,5 +442,6 @@
         <axis xyz="0 0 1"/>
         <limit effort="1" velocity="20"/>
-        <joint_properties friction="0.0"/>
+        <!-- <joint_properties friction="0.0"/> -->
+        <xacro:gazebo_joints/>
     </joint>
     <joint name="right_passive_wheel_joint" type="continuous">
@@ -439,5 +451,6 @@
         <axis xyz="0 0 1"/>
         <limit effort="1" velocity="20"/>
-        <joint_properties friction="0.0"/>
+        <!-- <joint_properties friction="0.0"/> -->
+        <xacro:gazebo_joints/>
     </joint>
     <!-- <joint name="world_to_base_link" type="fixed">
@@ -471,5 +484,6 @@
         <axis xyz="0 0 1"/>
         <limit effort="1" velocity="20" />
-        <joint_properties friction="0.0"/>
+        <!-- <joint_properties friction="0.0"/> -->
+        <xacro:gazebo_joints/>
     </joint>
     <joint name="right_spinning_wheel" type="continuous">
@@ -479,5 +493,6 @@
         <axis xyz="0 0 1"/>
         <limit effort="1" velocity="20" />
-        <joint_properties friction="0.0"/>
+        <!-- <joint_properties friction="0.0"/> -->
+        <xacro:gazebo_joints/>
     </joint>
     <joint name="left_passive_wheel" type="continuous">
@@ -487,5 +502,6 @@
         <axis xyz="0 0 1"/>
         <limit effort="1" velocity="20" />
-        <joint_properties friction="0.0"/>
+        <!-- <joint_properties friction="0.0"/> -->
+        <xacro:gazebo_joints/>
     </joint>
     <joint name="right_passive_wheel" type="continuous">
@@ -495,5 +511,6 @@
         <axis xyz="0 0 1"/>
         <limit effort="1" velocity="20" />
-        <joint_properties friction="0.0"/>
+        <!-- <joint_properties friction="0.0"/> -->
+        <xacro:gazebo_joints/>
     </joint>
     <joint name="plow_to_base" type="revolute">
@@ -503,5 +520,6 @@
         <axis xyz="0 0 1"/>
         <limit effort="1" velocity="20" lower="0.2" upper="0" />
-        <joint_properties friction="0.0"/>
+        <!-- <joint_properties friction="0.0"/> -->
+        <xacro:gazebo_joints/>
     </joint>
     <!-- <joint name="slew" type="continuous">
@@ -519,5 +537,6 @@
         <axis xyz="0 0 1"/>
         <limit effort="1" velocity="20" />
-        <joint_properties friction="0.0"/>
+        <!-- <joint_properties friction="0.0"/> -->
+        <xacro:gazebo_joints/>
     </joint>
     <!-- <joint name="fixed_base" type="fixed">
@@ -535,5 +554,6 @@
         <axis xyz="0 0 1"/>
         <limit effort="1" velocity="20" lower="-1.2217304763960306069" upper="0.87266462599716476678"/>
-        <joint_properties friction="0.0"/>
+        <!-- <joint_properties friction="0.0"/> -->
+        <xacro:gazebo_joints/>
     </joint>
     <joint name="arm_to_boom" type="revolute">
@@ -543,5 +563,6 @@
         <axis xyz="0 0 1"/>
         <limit effort="1" velocity="20" lower="-0.5" upper="1.57"/>
-        <joint_properties friction="0.0"/>
+        <!-- <joint_properties friction="0.0"/> -->
+        <xacro:gazebo_joints/>
     </joint>
     <joint name="boom_to_swing" type="revolute">
@@ -551,5 +572,6 @@
         <axis xyz="0 0 1"/>
         <limit effort="1" velocity="20" lower="-0.4" upper="0.4" />
-        <joint_properties friction="0.0"/>
+        <!-- <joint_properties friction="0.0"/> -->
+        <xacro:gazebo_joints/>
     </joint>
     <joint name="swing_to_cabin" type="revolute">
@@ -559,7 +581,9 @@
         <axis xyz="0 0 1"/>
         <limit effort="1" velocity="20" lower="-1" upper="1.57" />
-        <joint_properties friction="0.0"/>
-    </joint>
-    <gravity>1</gravity>
+        <!-- <joint_properties friction="0.0"/> -->
+        <xacro:gazebo_joints/>
+    </joint>
+    <!-- <gravity>1</gravity> -->
+<!--
     <ros2_control name="GazeboSystem" type="system">
         <hardware>
@@ -567,9 +591,35 @@
         </hardware>
         <joint name="head_swivel" />
-    </ros2_control>
+    </ros2_control> -->
     <gazebo>
-        <plugin filename="libgazebo_ros2_control.so" name="gazebo_ros2_control">
-            <parameters>$(find urdf_visualize)/config/09a-minimal.yaml</parameters>
-        </plugin>
+        <plugin name='skid_steer_drive' filename='libgazebo_ros_diff_drive.so'>
+        <ros>
+          <!-- <namespace>/demo</namespace> -->
+          <argument>cmd_vel:=cmd_demo</argument>
+          <!-- <argument>odom:=odom</argument> -->
+        </ros>
+        <!-- Number of wheel pairs -->
+        <num_wheel_pairs>2</num_wheel_pairs>
+        <!-- wheels0 -->
+        <left_joint>wheel_left_spinning</left_joint>
+        <right_joint>wheel_left_free</right_joint>
+        <!-- wheels1-->
+        <left_joint>wheel_right_spinning</left_joint>
+        <right_joint>wheel_right_free</right_joint>
+        <!-- kinematics -->
+        <wheel_separation>1.748</wheel_separation>
+        <wheel_separation>1.748</wheel_separation>
+        <wheel_diameter>${wheel_radius*2}</wheel_diameter>
+        <wheel_diameter>${wheel_radius*2}</wheel_diameter>
+        <!-- limits -->
+        <max_wheel_torque>500</max_wheel_torque>
+        <max_wheel_acceleration>1.0</max_wheel_acceleration>
+        <!-- output -->
+        <publish_odom>true</publish_odom>
+        <publish_odom_tf>true</publish_odom_tf>
+        <publish_wheel_tf>true</publish_wheel_tf>
+        <odometry_frame>odom</odometry_frame>
+        <robot_base_frame>base_link</robot_base_frame>
+      </plugin>
     </gazebo>
 </robot>

Commit message: gazebo_ros2_control intro

File: urdf_visualize/urdf/robot.urdf (robot description, URDF)
Before this commit: robot onshape, 16 links, 15 joints
Links:
- link arm_base: geometry collision mesh filename=file:///home/christoa/nav2_ws/install/urdf_visualize/share/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; visual mesh filename=file:///home/christoa/nav2_ws/install/urdf_visualize/share/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
- link boom_base: geometry collision mesh filename=file:///home/christoa/nav2_ws/install/urdf_visualize/share/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; visual mesh filename=file:///home/christoa/nav2_ws/install/urdf_visualize/share/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
- link bucket_base: geometry collision mesh filename=file:///home/christoa/nav2_ws/install/urdf_visualize/share/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; collision mesh filename=file:///home/christoa/nav2_ws/install/urdf_visualize/share/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
- link cabin_base: geometry collision mesh filename=file:///home/christoa/nav2_ws/install/urdf_visualize/share/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; visual mesh filename=file:///home/christoa/nav2_ws/install/urdf_visualize/share/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
- link left_front_wheel_link: geometry collision mesh filename=file:///home/christoa/nav2_ws/install/urdf_visualize/share/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; visual mesh filename=file:///home/christoa/nav2_ws/install/urdf_visualize/share/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
- link left_spinning_wheel_link: geometry collision mesh filename=file:///home/christoa/nav2_ws/install/urdf_visualize/share/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; visual mesh filename=file:///home/christoa/nav2_ws/install/urdf_visualize/share/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
- link push_blade_bucket: geometry collision mesh filename=file:///home/christoa/nav2_ws/install/urdf_visualize/share/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; visual mesh filename=file:///home/christoa/nav2_ws/install/urdf_visualize/share/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
- link right_front_wheel_link: geometry collision mesh filename=file:///home/christoa/nav2_ws/install/urdf_visualize/share/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; visual mesh filename=file:///home/christoa/nav2_ws/install/urdf_visualize/share/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
- link right_spinning_wheel_link: geometry collision mesh filename=file:///home/christoa/nav2_ws/install/urdf_visualize/share/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; visual mesh filename=file:///home/christoa/nav2_ws/install/urdf_visualize/share/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
- link swing_base: geometry collision mesh filename=file:///home/christoa/nav2_ws/install/urdf_visualize/share/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; visual mesh filename=file:///home/christoa/nav2_ws/install/urdf_visualize/share/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
- link turret_base: geometry collision mesh filename=file:///home/christoa/nav2_ws/install/urdf_visualize/share/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; visual mesh filename=file:///home/christoa/nav2_ws/install/urdf_visualize/share/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
Joints:
- joint slew: origin xyz=0 0 0 rpy=-5.5511151231419568159e-17 -1.1102230246202266528e-16 -3.1415 -> xyz=0 0 0.1 rpy=-5.5511151231419568159e-17 -1.1102230246202266528e-16 -3.1415

File: urdf_visualize/urdf/robot_wheel.xacro (robot description, xacro)
@@ -410,11 +410,10 @@
     </link>
     <xacro:macro name="gazebo_joints">
-        <!-- <gazebo>
+        <gazebo>
             <joint>
                 <stiffness>100000.0</stiffness>
-                <damping>5</damping>
+                <damping>1000</damping>
             </joint>
         </gazebo>
-        <joint_properties damping="5" friction="0.9"/> -->
     </xacro:macro>
     <joint name="left_spinning_wheel_joint" type="continuous">
@@ -532,9 +531,9 @@
     </joint> -->
     <joint name="slew" type="continuous">
-        <origin xyz="0 0 0" rpy="-5.5511151231419568159e-17 -1.1102230246202266528e-16 -3.1415" />
+        <origin xyz="0 0 0.1" rpy="-5.5511151231419568159e-17 -1.1102230246202266528e-16 -3.1415" />
         <parent link="turret_base" />
         <child link="cabin_base" />
         <axis xyz="0 0 1"/>
-        <limit effort="1" velocity="20" />
+        <limit effort="1000" velocity="1" />
         <!-- <joint_properties friction="0.0"/> -->
         <xacro:gazebo_joints/>
@@ -571,5 +570,5 @@
         <child link="boom_base" />
         <axis xyz="0 0 1"/>
-        <limit effort="1" velocity="20" lower="-0.4" upper="0.4" />
+        <limit effort="1000" velocity="1" lower="-0.4" upper="0.4" />
         <!-- <joint_properties friction="0.0"/> -->
         <xacro:gazebo_joints/>
@@ -585,41 +584,38 @@
     </joint>
     <!-- <gravity>1</gravity> -->
-<!--
     <ros2_control name="GazeboSystem" type="system">
-        <hardware>
-            <plugin>gazebo_ros2_control/GazeboSystem</plugin>
-        </hardware>
-        <joint name="head_swivel" />
-    </ros2_control> -->
+    <hardware>
+        <plugin>gazebo_ros2_control/GazeboSystem</plugin>
+    </hardware>
+    <joint name="slew">
+        <!-- <param name="pos_kp">10</param>
+        <param name="pos_ki">1</param>
+        <param name="pos_kd">2</param>
+        <param name="pos_max_integral_error">10000</param>
+        <param name="vel_kp">10</param>
+        <param name="vel_ki">5</param>
+        <param name="vel_kd">2</param>
+        <param name="vel_max_integral_error">10000</param> -->
+        <command_interface name="effort"/>
+        <!-- <command_interface name="velocity_pid"/> -->
+        <state_interface name="position">
+        </state_interface>
+        <state_interface name="velocity"/>
+        <state_interface name="effort"/>
+    </joint>
+    <joint name="boom_to_swing">
+        <command_interface name="effort"/>
+        <state_interface name="position">
+        </state_interface>
+        <state_interface name="velocity"/>
+        <state_interface name="effort"/>
+    </joint>
+    </ros2_control>
     <gazebo>
-        <plugin name='skid_steer_drive' filename='libgazebo_ros_diff_drive.so'>
-        <ros>
-          <!-- <namespace>/demo</namespace> -->
-          <argument>cmd_vel:=cmd_demo</argument>
-          <!-- <argument>odom:=odom</argument> -->
-        </ros>
-        <!-- Number of wheel pairs -->
-        <num_wheel_pairs>2</num_wheel_pairs>
-        <!-- wheels0 -->
-        <left_joint>wheel_left_spinning</left_joint>
-        <right_joint>wheel_left_free</right_joint>
-        <!-- wheels1-->
-        <left_joint>wheel_right_spinning</left_joint>
-        <right_joint>wheel_right_free</right_joint>
-        <!-- kinematics -->
-        <wheel_separation>1.748</wheel_separation>
-        <wheel_separation>1.748</wheel_separation>
-        <wheel_diameter>${wheel_radius*2}</wheel_diameter>
-        <wheel_diameter>${wheel_radius*2}</wheel_diameter>
-        <!-- limits -->
-        <max_wheel_torque>500</max_wheel_torque>
-        <max_wheel_acceleration>1.0</max_wheel_acceleration>
-        <!-- output -->
-        <publish_odom>true</publish_odom>
-        <publish_odom_tf>true</publish_odom_tf>
-        <publish_wheel_tf>true</publish_wheel_tf>
-        <odometry_frame>odom</odometry_frame>
-        <robot_base_frame>base_link</robot_base_frame>
-      </plugin>
+        <plugin filename="libgazebo_ros2_control.so" name="gazebo_ros2_control">
+            <robot_param>robot_description</robot_param>
+            <robot_param_node>robot_state_publisher</robot_param_node>
+            <parameters>$(find sambot_description)/params/ros2_controllers.yaml</parameters>
+        </plugin>
     </gazebo>
 </robot>
