Commit message: added proper control launch instead of the nav2 frankenstein

File: urdf_visualize/urdf/robot.urdf (robot description, URDF)
Before this commit: robot onshape, 16 links, 15 joints
Links:
- removed link wheel_left_free
- removed link wheel_left_spinning
- removed link wheel_right_free
- removed link wheel_right_spinning
- added link left_skid_wheel_free, mass 43.19562500000001; collision cylinder length=0.2 radius=0.25; visual cylinder length=0.2 radius=0.25
- added link left_skid_wheel_spinning, mass 43.19562500000001; collision cylinder length=0.2 radius=0.25; visual cylinder length=0.2 radius=0.25
- added link right_skid_wheel_free, mass 43.19562500000001; collision cylinder length=0.2 radius=0.25; visual cylinder length=0.2 radius=0.25
- added link right_skid_wheel_spinning, mass 43.19562500000001; collision cylinder length=0.2 radius=0.25; visual cylinder length=0.2 radius=0.25
Joints:
- removed joint left_passive_wheel_joint
- removed joint left_spinning_wheel_joint
- removed joint right_passive_wheel_joint
- removed joint right_spinning_wheel_joint
- added joint left_free_to_skid: type fixed, parent left_front_wheel_link, child left_skid_wheel_free, origin xyz=0 0 0.3 rpy=0 0 0, axis 0 0 1
- added joint left_spin_to_skid: type fixed, parent left_spinning_wheel_link, child left_skid_wheel_spinning, origin xyz=0 0 -0.3 rpy=0 0 0, axis 0 0 1
- added joint right_free_to_skid: type fixed, parent right_front_wheel_link, child right_skid_wheel_free, origin xyz=0 0 -0.3 rpy=0 0 0, axis 0 0 1, limit effort=1000 velocity=1
- added joint right_spin_to_skid: type fixed, parent right_spinning_wheel_link, child right_skid_wheel_spinning, origin xyz=0 0 -0.3 rpy=0 0 0, axis 0 0 1
- joint arm_to_boom: limit lower=-0.5 upper=1.57 effort=1 velocity=20 -> lower=-0.5 upper=1.57 effort=1000 velocity=1
- joint boom_to_swing: limit lower=-0.4 upper=0.4 effort=1 velocity=20 -> lower=-0.4 upper=0.4 effort=1000 velocity=1
- joint bucket_to_arm: limit lower=-1.2217304763960306069 upper=0.87266462599716476678 effort=1 velocity=20 -> lower=-1.2217304763960306069 upper=0.87266462599716476678 effort=1000 velocity=1
- joint left_passive_wheel: limit effort=1 velocity=20 -> effort=1000 velocity=1
- joint left_spinning_wheel: limit effort=1 velocity=20 -> effort=1000 velocity=1
- joint plow_to_base: limit lower=0.2 upper=0 effort=1 velocity=20 -> lower=0.2 upper=0 effort=1000 velocity=1
- joint right_passive_wheel: limit effort=1 velocity=20 -> effort=1000 velocity=1
- joint right_spinning_wheel: limit effort=1 velocity=20 -> effort=1000 velocity=1
- joint slew: limit effort=1 velocity=20 -> effort=1000 velocity=1
- joint swing_to_cabin: limit lower=-1 upper=1.57 effort=1 velocity=20 -> lower=-1 upper=1.57 effort=1000 velocity=1

File: urdf_visualize/urdf/robot_wheel.xacro (robot description, xacro)
@@ -294,5 +294,5 @@
     <xacro:property name="wheel_radius" value="0.25"/>
     <xacro:property name="wheel_length" value="0.2"/>
-    <xacro:property name="wheel_mass" value="${3.1415*(wheel_radius**2)*wheel_length*rubber_density}"/>
+    <xacro:property name="wheel_mass" value="${100*3.1415*(wheel_radius**2)*wheel_length*rubber_density}"/>
     <xacro:property name="wheel_ixx" value="${(1/12)*wheel_mass*(3*wheel_radius**2 + wheel_length**2)}"/>
     <xacro:property name="wheel_iyy" value="${(1/12)*wheel_mass*(3*wheel_radius**2 + wheel_length**2)}"/>
@@ -422,5 +422,5 @@
             <joint>
                 <stiffness>1000.0</stiffness>
-                <damping>5</damping>
+                <damping>500</damping>
             </joint>
         </gazebo>
@@ -501,5 +501,5 @@
         <xacro:gazebo_joints/>
     </joint>
-    <joint name="slew" type="continuous">
+    <joint name="excavator_slew" type="fixed">
         <origin xyz="0 0 0.1" rpy="-5.5511151231419568159e-17 -1.1102230246202266528e-16 -3.1415" />
         <parent link="turret_base" />
@@ -548,7 +548,5 @@
                 <param name="max">1000</param>
             </command_interface>
-            <state_interface name="position">
-                <param name="initial_value">0</param>
-            </state_interface>
+            <state_interface name="position"/>
             <state_interface name="velocity"/>
             <state_interface name="effort"/>
@@ -567,5 +565,5 @@
         </transmission>
     </xacro:macro>
-    <xacro:simple_transmission name="slew"/>
+    <xacro:simple_transmission name="excavator_slew"/>
     <xacro:simple_transmission name="plow_to_base"/>
     <xacro:simple_transmission name="arm_to_bucket"/>
@@ -577,5 +575,5 @@
         <plugin>gazebo_ros2_control/GazeboSystem</plugin>
     </hardware>
-    <xacro:gazebo_ros2_control_joints name="slew"/>
+    <xacro:gazebo_ros2_control_joints name="excavator_slew"/>
     <xacro:gazebo_ros2_control_joints name="plow_to_base"/>
     <xacro:gazebo_ros2_control_joints name="arm_to_bucket"/>
@@ -586,8 +584,5 @@
     <gazebo>
         <plugin filename="libgazebo_ros2_control.so" name="gazebo_ros2_control">
-            <robot_param>robot_description</robot_param>
-            <robot_param_node>robot_state_publisher</robot_param_node>
             <parameters>$(find sambot_description)/params/ros2_controllers.yaml</parameters>
-            <controller_manager_prefix_node_name>controller_manager</controller_manager_prefix_node_name>
         </plugin>
     </gazebo>
