Commit message: somewhat working skid-steer

File: urdf_visualize/urdf/robot_wheel.xacro (robot description, xacro)
@@ -422,5 +422,5 @@
         <child link="wheel_left_spinning"/>
         <axis xyz="0 0 1"/>
-        <limit effort="1" velocity="20"/>
+        <limit effort="1000" velocity="1"/>
         <!-- <joint_properties friction="0.0"/> -->
         <xacro:gazebo_joints/>
@@ -431,5 +431,5 @@
         <child link="wheel_left_free"/>
         <axis xyz="0 0 1"/>
-        <limit effort="1" velocity="20"/>
+        <limit effort="1000" velocity="1"/>
         <!-- <joint_properties friction="0.0"/> -->
         <xacro:gazebo_joints/>
@@ -440,5 +440,5 @@
         <child link="wheel_right_spinning"/>
         <axis xyz="0 0 1"/>
-        <limit effort="1" velocity="20"/>
+        <limit effort="1000" velocity="1"/>
         <!-- <joint_properties friction="0.0"/> -->
         <xacro:gazebo_joints/>
@@ -449,5 +449,5 @@
         <child link="wheel_right_free"/>
         <axis xyz="0 0 1"/>
-        <limit effort="1" velocity="20"/>
+        <limit effort="1000" velocity="1"/>
         <!-- <joint_properties friction="0.0"/> -->
         <xacro:gazebo_joints/>
@@ -475,5 +475,5 @@
         <child link="cabin_base" />
         <axis xyz="0 0 1"/>
-        <limit effort="1" velocity="20" />
+        <limit effort="1000" velocity="1" />
     </joint> -->
     <joint name="left_spinning_wheel" type="continuous">
@@ -482,5 +482,5 @@
         <child link="left_spinning_wheel_link" />
         <axis xyz="0 0 1"/>
-        <limit effort="1" velocity="20" />
+        <limit effort="1000" velocity="1" />
         <!-- <joint_properties friction="0.0"/> -->
         <xacro:gazebo_joints/>
@@ -491,5 +491,5 @@
         <child link="right_spinning_wheel_link" />
         <axis xyz="0 0 1"/>
-        <limit effort="1" velocity="20" />
+        <limit effort="1000" velocity="1" />
         <!-- <joint_properties friction="0.0"/> -->
         <xacro:gazebo_joints/>
@@ -500,5 +500,5 @@
         <child link="left_front_wheel_link" />
         <axis xyz="0 0 1"/>
-        <limit effort="1" velocity="20" />
+        <limit effort="1000" velocity="1" />
         <!-- <joint_properties friction="0.0"/> -->
         <xacro:gazebo_joints/>
@@ -509,5 +509,5 @@
         <child link="right_front_wheel_link" />
         <axis xyz="0 0 1"/>
-        <limit effort="1" velocity="20" />
+        <limit effort="1000" velocity="1" />
         <!-- <joint_properties friction="0.0"/> -->
         <xacro:gazebo_joints/>
@@ -518,5 +518,5 @@
         <child link="push_blade_bucket" />
         <axis xyz="0 0 1"/>
-        <limit effort="1" velocity="20" lower="0.2" upper="0" />
+        <limit effort="1000" velocity="1" lower="0.2" upper="0" />
         <!-- <joint_properties friction="0.0"/> -->
         <xacro:gazebo_joints/>
@@ -527,5 +527,5 @@
         <child link="turret_base" />
         <axis xyz="0 0 1"/>
-        <limit effort="1" velocity="20" />
+        <limit effort="1000" velocity="1" />
         <joint_properties friction="0.0"/>
     </joint> -->
@@ -544,5 +544,5 @@
         <child link="compact_excavator_turret_cabin_roller" />
         <axis xyz="0 0 1"/>
-        <limit effort="1" velocity="20" />
+        <limit effort="1000" velocity="1" />
         <joint_properties friction="0.0"/>
     </joint> -->
@@ -552,5 +552,5 @@
         <child link="bucket_base" />
         <axis xyz="0 0 1"/>
-        <limit effort="1" velocity="20" lower="-1.2217304763960306069" upper="0.87266462599716476678"/>
+        <limit effort="1000" velocity="1" lower="-1.2217304763960306069" upper="0.87266462599716476678"/>
         <!-- <joint_properties friction="0.0"/> -->
         <xacro:gazebo_joints/>
@@ -561,5 +561,5 @@
         <child link="arm_base" />
         <axis xyz="0 0 1"/>
-        <limit effort="1" velocity="20" lower="-0.5" upper="1.57"/>
+        <limit effort="1000" velocity="1" lower="-0.5" upper="1.57"/>
         <!-- <joint_properties friction="0.0"/> -->
         <xacro:gazebo_joints/>
@@ -579,5 +579,5 @@
         <child link="swing_base" />
         <axis xyz="0 0 1"/>
-        <limit effort="1" velocity="20" lower="-1" upper="1.57" />
+        <limit effort="1000" velocity="1" lower="-1" upper="1.57" />
         <!-- <joint_properties friction="0.0"/> -->
         <xacro:gazebo_joints/>
@@ -619,3 +619,32 @@
         </plugin>
     </gazebo>
+    <!-- skidsteer -->
+     <gazebo>
+    <plugin name="two_wheeled_robot_diff_drive" filename="libgazebo_ros_diff_drive.so">
+        <ros>
+        </ros>
+        <!-- Number of wheel pairs -->
+        <num_wheel_pairs>2</num_wheel_pairs>
+        <!-- TODO fix the link names -->
+        <!-- wheels0 -->
+        <left_joint>left_spinning_wheel_joint</left_joint>
+        <left_joint>left_passive_wheel_joint</left_joint>
+        <right_joint>right_spinning_wheel_joint</right_joint>
+        <right_joint>right_passive_wheel_joint</right_joint>
+        <!-- kinematics -->
+        <wheel_separation>1.25</wheel_separation>
+        <wheel_separation>1.25</wheel_separation>
+        <wheel_diameter>1.0</wheel_diameter>
+        <wheel_diameter>0.6</wheel_diameter>
+        <!-- limits -->
+        <max_wheel_torque>20</max_wheel_torque>
+        <max_wheel_acceleration>1.0</max_wheel_acceleration>
+        <!-- output -->
+        <publish_odom>true</publish_odom>
+        <publish_odom_tf>true</publish_odom_tf>
+        <publish_wheel_tf>true</publish_wheel_tf>
+        <odometry_frame>odom</odometry_frame>
+        <robot_base_frame>base_link</robot_base_frame>
+    </plugin>
+    </gazebo>
 </robot>

Commit message: fixed xacro

File: urdf_visualize/urdf/robot_wheel.xacro (robot description, xacro)
@@ -41,27 +41,4 @@
         </inertial>
     </link>
-<!--
-    <link name="turret_base">
-        <visual>
-            <origin xyz="1.232595164407830946e-32 8.7258015952359883014e-17 -0.11999999999999998168" rpy="0 0 0" />
-            <geometry>
-                <mesh filename="file://$(find urdf_visualize)/meshes/compact_excavator_frame_body.stl"/>
-            </geometry>
-                <material name="compact_excavator_frame_body_material">
-            <color rgba="0.91764705882352937127 0.91764705882352937127 0.91764705882352937127 1.0"/>
-            </material>
-        </visual>
-        <collision>
-            <origin xyz="1.232595164407830946e-32 8.7258015952359883014e-17 -0.11999999999999998168" rpy="0 0 0" />
-            <geometry>
-            <mesh filename="file://$(find urdf_visualize)/meshes/compact_excavator_frame_body.stl"/>
-            </geometry>
-        </collision>
-        <inertial>
-            <origin xyz="-0.0067641129059075200819 -0.12553013124423664792 -0.18649077363537946983" rpy="0 0 0"/>
-            <mass value="459.11707598787205598" />
-            <inertia ixx="103.54309263053609413" ixy="2.8689912175751035583"  ixz="-0.26918599165092144121" iyy="71.550382439979060223" iyz="-8.7881744003938315757" izz="164.71779214088334697" />
-        </inertial>
-    </link> -->
     <link name="turret_base">
         <visual>
@@ -321,5 +298,5 @@
     <xacro:property name="wheel_iyy" value="${(1/12)*wheel_mass*(3*wheel_radius**2 + wheel_length**2)}"/>
     <xacro:property name="wheel_izz" value="${(1/2)*wheel_mass*wheel_radius**2}"/>
-    <link name="wheel_left_spinning">
+    <link name="left_skid_wheel_spinning">
         <visual>
             <origin xyz="0 0 0" rpy="0 0 0"/>
@@ -337,4 +314,12 @@
             </geometry>
         </collision>
+        <surface>
+            <friction>
+                <ode>
+                    <mu>1</mu>
+                    <mu2>1</mu2>
+                </ode>
+            </friction>
+        </surface>
         <inertial>
             <origin xyz="0 0 0" rpy="0 0 0"/>
@@ -343,5 +328,5 @@
         </inertial>
     </link>
-    <link name="wheel_left_free">
+    <link name="left_skid_wheel_free">
         <visual>
             <origin xyz="0 0 0" rpy="0 0 0"/>
@@ -359,4 +344,12 @@
             </geometry>
         </collision>
+        <surface>
+            <friction>
+                <ode>
+                    <mu>1</mu>
+                    <mu2>1</mu2>
+                </ode>
+            </friction>
+        </surface>
         <inertial>
             <origin xyz="0 0 0" rpy="0 0 0"/>
@@ -365,5 +358,5 @@
         </inertial>
     </link>
-    <link name="wheel_right_spinning">
+    <link name="right_skid_wheel_spinning">
         <visual>
             <origin xyz="0 0 0" rpy="0 0 0"/>
@@ -381,4 +374,12 @@
             </geometry>
         </collision>
+        <surface>
+            <friction>
+                <ode>
+                    <mu>1</mu>
+                    <mu2>1</mu2>
+                </ode>
+            </friction>
+        </surface>
         <inertial>
             <origin xyz="0 0 0" rpy="0 0 0"/>
@@ -387,5 +388,5 @@
         </inertial>
     </link>
-    <link name="wheel_right_free">
+    <link name="right_skid_wheel_free">
         <visual>
             <origin xyz="0 0 0" rpy="0 0 0"/>
@@ -403,4 +404,12 @@
             </geometry>
         </collision>
+        <surface>
+            <friction>
+                <ode>
+                    <mu>1</mu>
+                    <mu2>1</mu2>
+                </ode>
+            </friction>
+        </surface>
         <inertial>
             <origin xyz="0 0 0" rpy="0 0 0"/>
@@ -412,50 +421,38 @@
         <gazebo>
             <joint>
-                <stiffness>100000.0</stiffness>
-                <damping>1000</damping>
+                <stiffness>1000.0</stiffness>
+                <damping>5</damping>
             </joint>
         </gazebo>
     </xacro:macro>
-    <joint name="left_spinning_wheel_joint" type="continuous">
+    <joint name="left_spin_to_skid" type="fixed">
         <origin xyz="0 0 -0.3" rpy="0 0 0"/>
         <parent link="left_spinning_wheel_link"/>
-        <child link="wheel_left_spinning"/>
-        <axis xyz="0 0 1"/>
-        <limit effort="1000" velocity="1"/>
-        <!-- <joint_properties friction="0.0"/> -->
-        <xacro:gazebo_joints/>
-    </joint>
-    <joint name="left_passive_wheel_joint" type="continuous">
+        <child link="left_skid_wheel_spinning"/>
+        <axis xyz="0 0 1"/>
+        <xacro:gazebo_joints/>
+    </joint>
+    <joint name="left_free_to_skid" type="fixed">
         <origin xyz="0 0 0.3" rpy="0 0 0"/>
         <parent link="left_front_wheel_link"/>
-        <child link="wheel_left_free"/>
-        <axis xyz="0 0 1"/>
-        <limit effort="1000" velocity="1"/>
-        <!-- <joint_properties friction="0.0"/> -->
-        <xacro:gazebo_joints/>
-    </joint>
-    <joint name="right_spinning_wheel_joint" type="continuous">
+        <child link="left_skid_wheel_free"/>
+        <axis xyz="0 0 1"/>
+        <xacro:gazebo_joints/>
+    </joint>
+    <joint name="right_spin_to_skid" type="fixed">
         <origin xyz="0 0 -0.3" rpy="0 0 0"/>
         <parent link="right_spinning_wheel_link"/>
-        <child link="wheel_right_spinning"/>
-        <axis xyz="0 0 1"/>
-        <limit effort="1000" velocity="1"/>
-        <!-- <joint_properties friction="0.0"/> -->
-        <xacro:gazebo_joints/>
-    </joint>
-    <joint name="right_passive_wheel_joint" type="continuous">
+        <child link="right_skid_wheel_spinning"/>
+        <axis xyz="0 0 1"/>
+        <xacro:gazebo_joints/>
+    </joint>
+    <joint name="right_free_to_skid" type="fixed">
         <origin xyz="0 0 -0.3" rpy="0 0 0"/>
         <parent link="right_front_wheel_link"/>
-        <child link="wheel_right_free"/>
+        <child link="right_skid_wheel_free"/>
         <axis xyz="0 0 1"/>
         <limit effort="1000" velocity="1"/>
-        <!-- <joint_properties friction="0.0"/> -->
-        <xacro:gazebo_joints/>
-    </joint>
-    <!-- <joint name="world_to_base_link" type="fixed">
-        <parent link="world"/>
-        <child link="base_link"/>
-        <origin xyz="0 0 0" rpy="0 0 0"/>
-    </joint> -->
+        <xacro:gazebo_joints/>
+    </joint>
     <joint name="base_to_turret" type="fixed">
         <origin xyz="0 0 0.55" rpy="0 0 0" />
@@ -464,17 +461,4 @@
         <axis xyz="0 0 1"/>
     </joint>
-    <!-- <joint name="base_to_cabin" type="fixed">
-        <origin xyz="0.15929227608280682738 -0.2512819772778476235 0.33139999999999991687" rpy="0 0 0" />
-        <parent link="base_link" />
-        <child link="cabin_base" />
-        <axis xyz="0 0 1"/>
-    </joint> -->
-    <!-- <joint name="turret_to_cabin" type="continuous">
-        <origin xyz="0 0 0" rpy="0 0 -3.142" />
-        <parent link="turret_base" />
-        <child link="cabin_base" />
-        <axis xyz="0 0 1"/>
-        <limit effort="1000" velocity="1" />
-    </joint> -->
     <joint name="left_spinning_wheel" type="continuous">
         <origin xyz="-0.5739999999999999547 -0.80000000000000015543 -0.2750000000000000222" rpy="1.570796326794896558 -0.3547477759675310427 1.5707963267948976682" />
@@ -483,5 +467,4 @@
         <axis xyz="0 0 1"/>
         <limit effort="1000" velocity="1" />
-        <!-- <joint_properties friction="0.0"/> -->
         <xacro:gazebo_joints/>
     </joint>
@@ -492,5 +475,4 @@
         <axis xyz="0 0 1"/>
         <limit effort="1000" velocity="1" />
-        <!-- <joint_properties friction="0.0"/> -->
         <xacro:gazebo_joints/>
     </joint>
@@ -501,5 +483,4 @@
         <axis xyz="0 0 1"/>
         <limit effort="1000" velocity="1" />
-        <!-- <joint_properties friction="0.0"/> -->
         <xacro:gazebo_joints/>
     </joint>
@@ -510,5 +491,4 @@
         <axis xyz="0 0 1"/>
         <limit effort="1000" velocity="1" />
-        <!-- <joint_properties friction="0.0"/> -->
         <xacro:gazebo_joints/>
     </joint>
@@ -519,15 +499,6 @@
         <axis xyz="0 0 1"/>
         <limit effort="1000" velocity="1" lower="0.2" upper="0" />
-        <!-- <joint_properties friction="0.0"/> -->
-        <xacro:gazebo_joints/>
-    </joint>
-    <!-- <joint name="slew" type="continuous">
-        <origin xyz="-0.25 -2.6052883279480892481e-15 -0.050000000000000002776" rpy="-5.5511151231419568159e-17 -1.1102230246202266528e-16 0" />
-        <parent link="compact_excavator_turret_cabin_roller" />
-        <child link="turret_base" />
-        <axis xyz="0 0 1"/>
-        <limit effort="1000" velocity="1" />
-        <joint_properties friction="0.0"/>
-    </joint> -->
+        <xacro:gazebo_joints/>
+    </joint>
     <joint name="slew" type="continuous">
         <origin xyz="0 0 0.1" rpy="-5.5511151231419568159e-17 -1.1102230246202266528e-16 -3.1415" />
@@ -536,16 +507,7 @@
         <axis xyz="0 0 1"/>
         <limit effort="1000" velocity="1" />
-        <!-- <joint_properties friction="0.0"/> -->
-        <xacro:gazebo_joints/>
-    </joint>
-    <!-- <joint name="fixed_base" type="fixed">
-        <origin xyz="-0.25 -2.394831672112794725e-15 0.049999999999999988898" rpy="-6.5400986663891116335e-25 -1.0029564927205460558e-23 3.1415926535897926719" />
-        <parent link="cabin_base" />
-        <child link="compact_excavator_turret_cabin_roller" />
-        <axis xyz="0 0 1"/>
-        <limit effort="1000" velocity="1" />
-        <joint_properties friction="0.0"/>
-    </joint> -->
-    <joint name="bucket_to_arm" type="revolute">
+        <xacro:gazebo_joints/>
+    </joint>
+    <joint name="arm_to_bucket" type="revolute">
         <origin xyz="0.12000000000000410338 -1.5403327562575612752 9.4368957093138305936e-16" rpy="3.1415926535897917837 1.8859935444767496044e-16 -1.5963552846072552871" />
         <parent link="arm_base" />
@@ -553,8 +515,7 @@
         <axis xyz="0 0 1"/>
         <limit effort="1000" velocity="1" lower="-1.2217304763960306069" upper="0.87266462599716476678"/>
-        <!-- <joint_properties friction="0.0"/> -->
-        <xacro:gazebo_joints/>
-    </joint>
-    <joint name="arm_to_boom" type="revolute">
+        <xacro:gazebo_joints/>
+    </joint>
+    <joint name="boom_to_arm" type="revolute">
         <origin xyz="-0.84000000000000030198 2.3549999999999999822 -0.13500000000000003664" rpy="3.1415926535897922278 6.9325343981756730312e-15 2.5555644018935783635" />
         <parent link="boom_base" />
@@ -562,8 +523,7 @@
         <axis xyz="0 0 1"/>
         <limit effort="1000" velocity="1" lower="-0.5" upper="1.57"/>
-        <!-- <joint_properties friction="0.0"/> -->
-        <xacro:gazebo_joints/>
-    </joint>
-    <joint name="boom_to_swing" type="revolute">
+        <xacro:gazebo_joints/>
+    </joint>
+    <joint name="swing_to_boom" type="revolute">
         <origin xyz="0.079999999999996157518 0.074999999999997291056 -0.1500000000000039635" rpy="-1.570796326794896558 0.39285813115170314935 -1.5707963267949009989" />
         <parent link="swing_base" />
@@ -571,8 +531,7 @@
         <axis xyz="0 0 1"/>
         <limit effort="1000" velocity="1" lower="-0.4" upper="0.4" />
-        <!-- <joint_properties friction="0.0"/> -->
-        <xacro:gazebo_joints/>
-    </joint>
-    <joint name="swing_to_cabin" type="revolute">
+        <xacro:gazebo_joints/>
+    </joint>
+    <joint name="cabin_to_swing" type="revolute">
         <origin xyz="-0.040707723917193447405 -0.80673603465099630316 0.38039999999999996039" rpy="3.141592653589793116 4.8797124238540929311e-17 0.21446312817660284633" />
         <parent link="cabin_base" />
@@ -580,35 +539,48 @@
         <axis xyz="0 0 1"/>
         <limit effort="1000" velocity="1" lower="-1" upper="1.57" />
-        <!-- <joint_properties friction="0.0"/> -->
         <xacro:gazebo_joints/>
     </joint>
     <!-- <gravity>1</gravity> -->
+    <xacro:macro name="gazebo_ros2_control_joints" params="name">
+        <joint name="${name}">
+            <command_interface name="effort">
+                <param name="min">-1000</param>
+                <param name="max">1000</param>
+            </command_interface>
+            <state_interface name="position">
+                <param name="initial_value">0</param>
+            </state_interface>
+            <state_interface name="velocity"/>
+            <state_interface name="effort"/>
+        </joint>
+    </xacro:macro>
+    <xacro:macro name="simple_transmission" params="name">
+        <transmission name="${name}_trans">
+            <type>transmission_interface/SimpleTransmission</type>
+            <joint name="${name}">
+            <hardwareInterface>effort</hardwareInterface>
+            </joint>
+            <actuator name="${name}_motor">
+            <hardwareInterface>effort</hardwareInterface>
+            <mechanicalReduction>1</mechanicalReduction>
+            </actuator>
+        </transmission>
+    </xacro:macro>
+    <xacro:simple_transmission name="slew"/>
+    <xacro:simple_transmission name="plow_to_base"/>
+    <xacro:simple_transmission name="arm_to_bucket"/>
+    <xacro:simple_transmission name="boom_to_arm"/>
+    <xacro:simple_transmission name="swing_to_boom"/>
+    <xacro:simple_transmission name="cabin_to_swing"/>
     <ros2_control name="GazeboSystem" type="system">
     <hardware>
         <plugin>gazebo_ros2_control/GazeboSystem</plugin>
     </hardware>
-    <joint name="slew">
-        <!-- <param name="pos_kp">10</param>
-        <param name="pos_ki">1</param>
-        <param name="pos_kd">2</param>
-        <param name="pos_max_integral_error">10000</param>
-        <param name="vel_kp">10</param>
-        <param name="vel_ki">5</param>
-        <param name="vel_kd">2</param>
-        <param name="vel_max_integral_error">10000</param> -->
-        <command_interface name="effort"/>
-        <!-- <command_interface name="velocity_pid"/> -->
-        <state_interface name="position">
-        </state_interface>
-        <state_interface name="velocity"/>
-        <state_interface name="effort"/>
-    </joint>
-    <joint name="boom_to_swing">
-        <command_interface name="effort"/>
-        <state_interface name="position">
-        </state_interface>
-        <state_interface name="velocity"/>
-        <state_interface name="effort"/>
-    </joint>
+    <xacro:gazebo_ros2_control_joints name="slew"/>
+    <xacro:gazebo_ros2_control_joints name="plow_to_base"/>
+    <xacro:gazebo_ros2_control_joints name="arm_to_bucket"/>
+    <xacro:gazebo_ros2_control_joints name="boom_to_arm"/>
+    <xacro:gazebo_ros2_control_joints name="swing_to_boom"/>
+    <xacro:gazebo_ros2_control_joints name="cabin_to_swing"/>
     </ros2_control>
     <gazebo>
@@ -617,34 +589,27 @@
             <robot_param_node>robot_state_publisher</robot_param_node>
             <parameters>$(find sambot_description)/params/ros2_controllers.yaml</parameters>
+            <controller_manager_prefix_node_name>controller_manager</controller_manager_prefix_node_name>
         </plugin>
     </gazebo>
     <!-- skidsteer -->
-     <gazebo>
-    <plugin name="two_wheeled_robot_diff_drive" filename="libgazebo_ros_diff_drive.so">
-        <ros>
-        </ros>
-        <!-- Number of wheel pairs -->
-        <num_wheel_pairs>2</num_wheel_pairs>
-        <!-- TODO fix the link names -->
-        <!-- wheels0 -->
-        <left_joint>left_spinning_wheel_joint</left_joint>
-        <left_joint>left_passive_wheel_joint</left_joint>
-        <right_joint>right_spinning_wheel_joint</right_joint>
-        <right_joint>right_passive_wheel_joint</right_joint>
-        <!-- kinematics -->
-        <wheel_separation>1.25</wheel_separation>
-        <wheel_separation>1.25</wheel_separation>
-        <wheel_diameter>1.0</wheel_diameter>
-        <wheel_diameter>0.6</wheel_diameter>
-        <!-- limits -->
-        <max_wheel_torque>20</max_wheel_torque>
-        <max_wheel_acceleration>1.0</max_wheel_acceleration>
-        <!-- output -->
-        <publish_odom>true</publish_odom>
-        <publish_odom_tf>true</publish_odom_tf>
-        <publish_wheel_tf>true</publish_wheel_tf>
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
Commit message: changed to continuous

File: urdf_visualize/urdf/robot_wheel.xacro (robot description, xacro)
@@ -501,5 +501,5 @@
         <xacro:gazebo_joints/>
     </joint>
-    <joint name="excavator_slew" type="fixed">
+    <joint name="excavator_slew" type="continuous">
         <origin xyz="0 0 0.1" rpy="-5.5511151231419568159e-17 -1.1102230246202266528e-16 -3.1415" />
         <parent link="turret_base" />
