Commit message: pre ignition stash

File: sambot_description/urdf/joints.xacro (robot description, xacro)
@@ -44,5 +44,5 @@
         <child link="${left_spinning_wheel_link_name}" />
         <axis xyz="0 0 1"/>
-        <limit effort="20000" velocity="5" />
+        <limit effort="1000" velocity="1" />
         <!-- <xacro:dynamics dyn_damping="0.1" dyn_friction="0.2"/> -->
     </joint>
@@ -52,5 +52,5 @@
         <child link="${right_spinning_wheel_link_name}" />
         <axis xyz="0 0 1"/>
-        <limit effort="20000" velocity="5" />
+        <limit effort="1000" velocity="1" />
         <!-- <xacro:dynamics dyn_damping="0.1" dyn_friction="0.2"/> -->
     </joint>
@@ -60,5 +60,5 @@
         <child link="${left_front_wheel_link_name}" />
         <axis xyz="0 0 1"/>
-        <limit effort="20000" velocity="5" />
+        <limit effort="1000" velocity="1" />
         <!-- <xacro:dynamics dyn_damping="0.1" dyn_friction="0.2"/> -->
     </joint>
@@ -68,5 +68,5 @@
         <child link="${right_front_wheel_link_name}" />
         <axis xyz="0 0 1"/>
-        <limit effort="20000" velocity="5" />
+        <limit effort="1000" velocity="1" />
         <!-- <xacro:dynamics dyn_damping="0.1" dyn_friction="0.2"/> -->
     </joint>
@@ -76,5 +76,5 @@
         <child link="${plow_link_name}" />
         <axis xyz="0 0 1"/>
-        <limit effort="20000" velocity="5" lower="0.2" upper="0" />
+        <limit effort="1000" velocity="1" lower="0.2" upper="0" />
         <!-- <xacro:dynamics dyn_damping="0.1" dyn_friction="0.2"/> -->
     </joint>
@@ -84,5 +84,5 @@
         <child link="${cabin_link_name}" />
         <axis xyz="0 0 1"/>
-        <limit effort="20000" velocity="5"/>
+        <limit effort="1000" velocity="1"/>
         <!-- <xacro:dynamics dyn_damping="0.1" dyn_friction="0.2"/> -->
     </joint>
@@ -92,5 +92,5 @@
         <child link="bucket_base" />
         <axis xyz="0 0 1"/>
-        <limit effort="20000" velocity="5" lower="-1.2217304763960306069" upper="0.87266462599716476678"/>
+        <limit effort="1000" velocity="1" lower="-1.2217304763960306069" upper="0.87266462599716476678"/>
         <!-- <xacro:dynamics dyn_damping="0.1" dyn_friction="0.2"/> -->
     </joint>
@@ -100,5 +100,5 @@
         <child link="${arm_link_name}" />
         <axis xyz="0 0 1"/>
-        <limit effort="20000" velocity="5" lower="-0.5" upper="1.57"/>
+        <limit effort="1000" velocity="1" lower="-0.5" upper="1.57"/>
         <!-- <xacro:dynamics dyn_damping="0.1" dyn_friction="0.2"/> -->
     </joint>
@@ -108,5 +108,5 @@
         <child link="${boom_link_name}" />
         <axis xyz="0 0 1"/>
-        <limit effort="20000" velocity="1.0" lower="-0.4" upper="1" />
+        <limit effort="1000" velocity="1.0" lower="-0.4" upper="1" />
         <!-- <xacro:dynamics dyn_damping="0.1" dyn_friction="0.2"/> -->
     </joint>
@@ -116,5 +116,5 @@
         <child link="${swing_link_name}" />
         <axis xyz="0 0 1"/>
-        <limit effort="20000" velocity="5" lower="-0.1" upper="0.1" />
+        <limit effort="1000" velocity="1" lower="-0.1" upper="0.1" />
         <!-- <xacro:dynamics dyn_damping="0.1" dyn_friction="0.2"/> -->
     </joint>

File: sambot_description/urdf/position/dynamics.xacro (robot description, xacro)
@@ -82,5 +82,5 @@
                 <plugin>gazebo_ros2_control/GazeboSystem</plugin>
             </hardware>
-            <xacro:gazebo_ros2_control_joints_effort name="${excavator_slew_joint_name}" effort_lim="20000"/>
+            <!-- <xacro:gazebo_ros2_control_joints_effort name="${excavator_slew_joint_name}" effort_lim="20000"/>
             <xacro:gazebo_ros2_control_joints_effort name="${cabin_to_swing_joint_name}"  effort_lim="20000"/>
             <xacro:gazebo_ros2_control_joints_effort name="${swing_to_boom_joint_name}"  effort_lim="20000"/>
@@ -93,5 +93,5 @@
             <xacro:gazebo_ros2_control_joints_velocity name="${boom_to_arm_joint_name}"  velocity_lim="1.0"/>
             <xacro:gazebo_ros2_control_joints_velocity name="${swing_to_boom_joint_name}"  velocity_lim="1.0"/>
-            <xacro:gazebo_ros2_control_joints_velocity name="${cabin_to_swing_joint_name}"  velocity_lim="1.0"/>
+            <xacro:gazebo_ros2_control_joints_velocity name="${cabin_to_swing_joint_name}"  velocity_lim="1.0"/> -->
             <xacro:gazebo_ros2_control_joints_position name="${excavator_slew_joint_name}" position_lim="${pi}"/>
             <xacro:gazebo_ros2_control_joints_position name="${cabin_to_swing_joint_name}"  position_lim="${pi}"/>
@@ -103,5 +103,5 @@
         <gazebo>
             <plugin name="gazebo_ros2_control" filename="libgazebo_ros2_control.so">
-                <parameters>$(find sambot_description)/params/ros2_controllers.yaml</parameters>
+                <parameters>$(find sambot_description)/params/position_controller.yaml</parameters>
             </plugin>
         </gazebo>

File: sambot_description/urdf/velocity/dynamics.xacro (robot description, xacro)
@@ -6,10 +6,10 @@
             <stiffness>${stiffness}</stiffness>
             <damping>${damping}</damping>
-            <pid>
-                <p>100</p>
+            <!-- <pid>
+                <p>1</p>
                 <i>0</i>
-                <d>0.1</d>
-            </pid>
-            <!-- <dynamics damping="0.1" friction="0.2"/> -->
+                <d>0</d>
+            </pid> -->
+            <dynamics damping="5000" friction="0.2"/>
         </gazebo>
     </xacro:macro>
@@ -61,14 +61,14 @@
         </transmission>
     </xacro:macro>
-    <xacro:gazebo_joint_dynamics joint_name="${excavator_slew_joint_name}" stiffness="1000" damping="0.1"/>
-    <xacro:gazebo_joint_dynamics joint_name="${plow_to_base_joint_name}" stiffness="1000" damping="0.1"/>
-    <xacro:gazebo_joint_dynamics joint_name="${arm_to_bucket_joint_name}" stiffness="10000" damping="500"/>
-    <xacro:gazebo_joint_dynamics joint_name="${boom_to_arm_joint_name}" stiffness="1000" damping="0.1"/>
-    <xacro:gazebo_joint_dynamics joint_name="${swing_to_boom_joint_name}" stiffness="1000" damping="0.1"/>
-    <xacro:gazebo_joint_dynamics joint_name="${cabin_to_swing_joint_name}" stiffness="1000" damping="0.1"/>
-    <xacro:gazebo_joint_dynamics joint_name="${left_spin_to_skid_joint_name}" stiffness="1000" damping="0.1"/>
-    <xacro:gazebo_joint_dynamics joint_name="${left_free_to_skid_joint_name}" stiffness="1000" damping="0.1"/>
-    <xacro:gazebo_joint_dynamics joint_name="${right_spin_to_skid_joint_name}" stiffness="1000" damping="0.1"/>
-    <xacro:gazebo_joint_dynamics joint_name="${right_free_to_skid_joint_name}" stiffness="1000" damping="0.1"/>
+    <xacro:gazebo_joint_dynamics joint_name="${excavator_slew_joint_name}" stiffness="30000" damping="5"/>
+    <xacro:gazebo_joint_dynamics joint_name="${plow_to_base_joint_name}" stiffness="30000" damping="5"/>
+    <xacro:gazebo_joint_dynamics joint_name="${arm_to_bucket_joint_name}" stiffness="30000" damping="5"/>
+    <xacro:gazebo_joint_dynamics joint_name="${boom_to_arm_joint_name}" stiffness="30000" damping="5"/>
+    <xacro:gazebo_joint_dynamics joint_name="${swing_to_boom_joint_name}" stiffness="30000" damping="5"/>
+    <xacro:gazebo_joint_dynamics joint_name="${cabin_to_swing_joint_name}" stiffness="30000" damping="5"/>
+    <xacro:gazebo_joint_dynamics joint_name="${left_spin_to_skid_joint_name}" stiffness="30000" damping="5"/>
+    <xacro:gazebo_joint_dynamics joint_name="${left_free_to_skid_joint_name}" stiffness="30000" damping="5"/>
+    <xacro:gazebo_joint_dynamics joint_name="${right_spin_to_skid_joint_name}" stiffness="30000" damping="5"/>
+    <xacro:gazebo_joint_dynamics joint_name="${right_free_to_skid_joint_name}" stiffness="30000" damping="5"/>
     <xacro:simple_transmission name="${excavator_slew_joint_name}"/>
     <xacro:simple_transmission name="${plow_to_base_joint_name}"/>
@@ -82,10 +82,10 @@
                 <plugin>gazebo_ros2_control/GazeboSystem</plugin>
             </hardware>
-            <xacro:gazebo_ros2_control_joints_effort name="${excavator_slew_joint_name}" effort_lim="20000"/>
+            <!-- <xacro:gazebo_ros2_control_joints_effort name="${excavator_slew_joint_name}" effort_lim="20000"/>
             <xacro:gazebo_ros2_control_joints_effort name="${cabin_to_swing_joint_name}"  effort_lim="20000"/>
             <xacro:gazebo_ros2_control_joints_effort name="${swing_to_boom_joint_name}"  effort_lim="20000"/>
             <xacro:gazebo_ros2_control_joints_effort name="${arm_to_bucket_joint_name}"  effort_lim="20000"/>
             <xacro:gazebo_ros2_control_joints_effort name="${boom_to_arm_joint_name}"  effort_lim="20000"/>
-            <xacro:gazebo_ros2_control_joints_effort name="${plow_to_base_joint_name}"  effort_lim="20000"/>
+            <xacro:gazebo_ros2_control_joints_effort name="${plow_to_base_joint_name}"  effort_lim="20000"/> -->
             <xacro:gazebo_ros2_control_joints_velocity name="${excavator_slew_joint_name}" velocity_lim="1.0"/>
             <xacro:gazebo_ros2_control_joints_velocity name="${plow_to_base_joint_name}"  velocity_lim="1.0"/>
@@ -94,4 +94,5 @@
             <xacro:gazebo_ros2_control_joints_velocity name="${swing_to_boom_joint_name}"  velocity_lim="1.0"/>
             <xacro:gazebo_ros2_control_joints_velocity name="${cabin_to_swing_joint_name}"  velocity_lim="1.0"/>
+<!--
             <xacro:gazebo_ros2_control_joints_position name="${excavator_slew_joint_name}" position_lim="${pi}"/>
             <xacro:gazebo_ros2_control_joints_position name="${cabin_to_swing_joint_name}"  position_lim="${pi}"/>
@@ -99,9 +100,9 @@
             <xacro:gazebo_ros2_control_joints_position name="${arm_to_bucket_joint_name}"  position_lim="${pi}"/>
             <xacro:gazebo_ros2_control_joints_position name="${boom_to_arm_joint_name}"  position_lim="${pi}"/>
-            <xacro:gazebo_ros2_control_joints_position name="${plow_to_base_joint_name}"  position_lim="${pi}"/>
+            <xacro:gazebo_ros2_control_joints_position name="${plow_to_base_joint_name}"  position_lim="${pi}"/> -->
         </ros2_control>
         <gazebo>
             <plugin name="gazebo_ros2_control" filename="libgazebo_ros2_control.so">
-                <parameters>$(find sambot_description)/params/ros2_controllers.yaml</parameters>
+                <parameters>$(find sambot_description)/params/velocity_controller.yaml</parameters>
             </plugin>
         </gazebo>
