Commit message: split main xacro into sub files

File: sambot_description/urdf/params.xacro (robot description, xacro)
@@ -18,3 +18,123 @@
     <xacro:property name="turret_base_material" value="0.9176 0.9176 0.9176 1.0"/>
     <xacro:property name="turret_base_inertial" value="103.54309263053609413 2.8689912175751035583 -0.26918599165092144121 71.550382439979060223 -8.7881744003938315757 164.71779214088334697"/>
+    <xacro:property name="left_spinning_wheel_link_mesh" value="${mesh_root}/compact_excavator_main_drive_wheel.stl"/>
+    <xacro:property name="left_spinning_wheel_link_origin" value="0 -2.0816681711721685133e-17 -0.015000000000000124345"/>
+    <xacro:property name="left_spinning_wheel_link_rpy" value="-4.71 0 0"/>
+    <xacro:property name="left_spinning_wheel_link_material" value="0.91764705882352937127 0.91764705882352937127 0.91764705882352937127 1.0"/>
+    <xacro:property name="left_spinning_wheel_link_inertial_origin" value="2.7929494467705319618e-05 -2.4226277708340838271e-16 -0.047030821852304713349"/>
+    <xacro:property name="left_spinning_wheel_link_inertial_rpy" value="0 0 0"/>
+    <xacro:property name="left_spinning_wheel_link_mass" value="35.986291345795820007"/>
+    <xacro:property name="left_spinning_wheel_link_inertial" value="0.20071737580058110484 2.1151248144254331483e-17 7.9696042408110000254e-05 0.20066206838835709547 2.9623558171777900037e-16 0.29333573070696433716"/>
+    <xacro:property name="right_spinning_wheel_link_mesh" value="${mesh_root}/compact_excavator_main_drive_wheel.stl"/>
+    <xacro:property name="right_spinning_wheel_link_origin" value="-6.9388939039072283776e-18 0 -0.015000000000000013323"/>
+    <xacro:property name="right_spinning_wheel_link_rpy" value="1.57 0 0"/>
+    <xacro:property name="right_spinning_wheel_link_material" value="0.91764705882352937127 0.91764705882352937127 0.91764705882352937127 1.0"/>
+    <xacro:property name="right_spinning_wheel_link_inertial_origin" value="2.7929494467698390888e-05 -2.2144767850277592569e-16 -0.047030821852304602326"/>
+    <xacro:property name="right_spinning_wheel_link_inertial_rpy" value="0 0 0"/>
+    <xacro:property name="right_spinning_wheel_link_mass" value="35.986291345795820007"/>
+    <xacro:property name="right_spinning_wheel_link_inertial" value="0.20071737580058127137 6.1250580134766935832e-18 7.9696042408110027359e-05 0.20066206838835703996 2.9623106429686494369e-16 0.29333573070696433716"/>
+    <xacro:property name="left_front_wheel_link_mesh" value="${mesh_root}/compact_excavator_front_wheel.stl"/>
+    <xacro:property name="left_front_wheel_link_origin" value="1.1102230246251565404e-16 -1.1102230246251565404e-16 -0.032500000000000084377"/>
+    <xacro:property name="left_front_wheel_link_rpy" value="0 1.570796326794896336 0"/>
+    <xacro:property name="left_front_wheel_link_material" value="0.91764705882352937127 0.91764705882352937127 0.91764705882352937127 1.0"/>
+    <xacro:property name="left_front_wheel_link_inertial_origin" value="8.8979772495497043726e-17 -1.1262368284473494847e-16 -0.032500000000000070499"/>
+    <xacro:property name="left_front_wheel_link_inertial_rpy" value="0 0 0"/>
+    <xacro:property name="left_front_wheel_link_mass" value="17.64673591392957519"/>
+    <xacro:property name="left_front_wheel_link_inertial" value="0.153078316536178205 1.0629206596102168903e-17 2.6922495826861160064e-17 0.15307831653617814949 6.9747558075870228735e-33 0.29963755764746907717"/>
+    <xacro:property name="right_front_wheel_link_mesh" value="${mesh_root}/compact_excavator_front_wheel.stl"/>
+    <xacro:property name="right_front_wheel_link_origin" value="-2.7755575615628913511e-17 0 -0.032500000000000084377"/>
+    <xacro:property name="right_front_wheel_link_rpy" value="-3.14 -1.570796326794896336 0"/>
+    <xacro:property name="right_front_wheel_link_material" value="0.91764705882352937127 0.91764705882352937127 0.91764705882352937127 1.0"/>
+    <xacro:property name="right_front_wheel_link_inertial_origin" value="-2.7755575615628913511e-17 0 -0.032500000000000084377"/>
+    <xacro:property name="right_front_wheel_link_inertial_rpy" value="0 0 0"/>
+    <xacro:property name="right_front_wheel_link_mass" value="17.64673591392957519"/>
+    <xacro:property name="right_front_wheel_link_inertial" value="0.153078316536178205 -1.0629206596102168903e-17 2.6922495826861160064e-17 0.15307831653617814949 6.9747558075870228735e-33 0.29963755764746907717"/>
+    <xacro:property name="push_blade_base_mesh" value="${mesh_root}/push_blade_bucket.stl"/>
+    <xacro:property name="push_blade_base_origin" value="-0.021564399534920564161 1.0799900599760599018 -0.25500000000000000444"/>
+    <xacro:property name="push_blade_base_rpy" value="-3.14 -1.57 0"/>
+    <xacro:property name="push_blade_base_material" value="0.61568627450980395466 0.81176470588235294379 0.92941176470588238168 1.0"/>
+    <xacro:property name="push_blade_base_inertial_origin" value="-0.10970493109347190241 0.88075063461342828486 -0.25500033703320834633"/>
+    <xacro:property name="push_blade_base_inertial_rpy" value="0 0 0"/>
+    <xacro:property name="push_blade_base_mass" value="147.01808168083425699"/>
+    <xacro:property name="push_blade_base_inertial" value="31.881096131626421197 0.91247385061899932701 -1.6212090668492922982e-05 21.196220352263214437 4.9900082202379639952e-06 13.169227707961496776"/>
+    <xacro:property name="swing_base_mesh" value="${mesh_root}/part01_pin_1.stl"/>
+    <xacro:property name="swing_base_origin" value="2.7755575615628913511e-17 0.074999999999999955591 -0.14999999999999996669"/>
+    <xacro:property name="swing_base_rpy" value="-3.14 -6.1629758220391547298e-33 -3.9110122218931175387e-17"/>
+    <xacro:property name="swing_base_material" value="0.61568627450980395466 0.81176470588235294379 0.92941176470588238168 1.0"/>
+    <xacro:property name="swing_base_inertial_origin" value="-0.026030309007671018073 0.10672288733099301317 0.097553850513847364945"/>
+    <xacro:property name="swing_base_inertial_rpy" value="0 0 0"/>
+    <xacro:property name="swing_base_mass" value="98.140190062279060612"/>
+    <xacro:property name="swing_base_inertial" value="2.6085778666185075458 0.040227300901953748358 0.42136783119553594679 3.1665232143977135593 -0.15916376835413623136 1.7889951810686841593"/>
+    <xacro:property name="boom_base_mesh" value="${mesh_root}/part02.stl"/>
+    <xacro:property name="boom_base_origin" value="0 -1.1102230246251565404e-16 -0.079999999999999987788"/>
+    <xacro:property name="boom_base_rpy" value="-1.57 0 0"/>
+    <xacro:property name="boom_base_material" value="0.77647058823529413463 0.7568627450980391913 0.73725490196078435901 1.0"/>
+    <xacro:property name="boom_base_inertial_origin" value="-0.04007940207094668611 1.215334476695421273 -0.079873417172118876817"/>
+    <xacro:property name="boom_base_inertial_rpy" value="0 0 0"/>
+    <xacro:property name="boom_base_mass" value="694.17793513858055121"/>
+    <xacro:property name="boom_base_inertial" value="242.81245205849677404 71.370938403077758494 0.0065905643878567711502 49.641340591529456105 -0.034260052091464154866 289.83702909122945357"/>
+    <xacro:property name="arm_base_mesh" value="${mesh_root}/part03.stl"/>
+    <xacro:property name="arm_base_origin" value="0 -2.2204460492503130808e-16 -0.054999999999999882316"/>
+    <xacro:property name="arm_base_rpy" value="1.57 0 0"/>
+    <xacro:property name="arm_base_material" value="0.98039215686274505668 0.71372549019607844922 0.0039215686274509803377 1.0"/>
+    <xacro:property name="arm_base_inertial_origin" value="0.10866226733951289685 -0.60164797350906107365 -0.055167291851018741833"/>
+    <xacro:property name="arm_base_inertial_rpy" value="0 0 0"/>
+    <xacro:property name="arm_base_mass" value="265.34907807560875881"/>
+    <xacro:property name="arm_base_inertial" value="57.599134249663784146 0.078442580554215754485 0.0049826290162324230956 1.8968981412117758012 0.02459901605653430981 58.868680211308259231"/>
+    <xacro:property name="bucket_link_name" value="bucket_base"/>
+    <xacro:property name="bucket_mesh1" value="${mesh_root}/part04.stl"/>
+    <xacro:property name="bucket_mesh1_origin" value="0.060000000000000053291 0.14000000000000012434 0.054999999999999993339"/>
+    <xacro:property name="bucket_mesh1_rpy" value="-3.14 -1.57 0"/>
+    <xacro:property name="bucket_mesh1_material" value="0.76862745098039220171 0.88627450980392152857 0.95294117647058818044 1.0"/>
+    <xacro:property name="bucket_mesh2" value="${mesh_root}/bucket.stl"/>
+    <xacro:property name="bucket_mesh2_origin" value="0.078718096856630614955 0.97961106773940276327 0.054999999999992416067"/>
+    <xacro:property name="bucket_mesh2_rpy" value="-1.57 0 3"/>
+    <xacro:property name="bucket_mesh2_material" value="0.61568627450980395466 0.81176470588235294379 0.92941176470588238168 1.0"/>
+    <xacro:property name="bucket_mesh3" value="${mesh_root}/bucket_mount.stl"/>
+    <xacro:property name="bucket_mesh3_origin" value="0.16999999999999237943 0.30800000000000604672 0.054999999999999299449"/>
+    <xacro:property name="bucket_mesh3_rpy" value="-4.71 -1.57 0"/>
+    <xacro:property name="bucket_mesh3_material" value="0.49803921568627451677 0.49803921568627451677 0.49803921568627451677 1.0"/>
+    <xacro:property name="bucket_inertial_origin" value="0.21363777998579594475 0.42618058483691984017 0.055071497454761988988"/>
+    <xacro:property name="bucket_inertial_rpy" value="0 0 0"/>
+    <xacro:property name="bucket_base_mass" value="132.70765933863819441"/>
+    <xacro:property name="bucket_base_inertial" value="14.03567187790122972 -1.6652440163767181502 0.0020270508814650067472 6.8549730106956987541 0.0040437120644442776929 11.610921270718170817"/>
+    <xacro:property name="rubber_density" value="1100"/>
+    <xacro:property name="wheel_radius" value="0.25"/>
+    <xacro:property name="wheel_length" value="0.2"/>
+    <xacro:macro name="skid_wheel" params="wheel_name mu1 mu2">
+        <xacro:property name="wheel_mass" value="${100*3.1415*(wheel_radius**2)*wheel_length*rubber_density}"/>
+        <xacro:property name="wheel_ixx" value="${(1/12)*wheel_mass*(3*wheel_radius**2 + wheel_length**2)}"/>
+        <xacro:property name="wheel_iyy" value="${(1/12)*wheel_mass*(3*wheel_radius**2 + wheel_length**2)}"/>
+        <xacro:property name="wheel_izz" value="${(1/2)*wheel_mass*wheel_radius**2}"/>
+        <link name="${wheel_name}">
+            <visual>
+                <origin xyz="0 0 0" rpy="0 0 0"/>
+                <geometry>
+                    <cylinder radius="${wheel_radius}" length="${wheel_length}"/>
+                </geometry>
+                <material name="wheel_material">
+                    <color rgba="0.5 0.5 0.5 1.0"/>
+                </material>
+            </visual>
+            <collision>
+                <origin xyz="0 0 0" rpy="0 0 0"/>
+                <geometry>
+                    <cylinder radius="${wheel_radius}" length="${wheel_length}"/>
+                </geometry>
+            </collision>
+            <surface>
+                <friction>
+                    <ode>
+                        <mu>${mu1}</mu>
+                        <mu2>${mu2}</mu2>
+                    </ode>
+                </friction>
+            </surface>
+            <inertial>
+                <origin xyz="0 0 0" rpy="0 0 0"/>
+                <mass value="${wheel_mass}"/>
+                <inertia ixx="${wheel_ixx}" ixy="0" ixz="0" iyy="${wheel_iyy}" iyz="0" izz="${wheel_izz}"/>
+            </inertial>
+        </link>
+    </xacro:macro>
 </robot>

Commit message: added meshes and comments

File: sambot_description/urdf/params.xacro (robot description, xacro)
@@ -1,5 +1,5 @@
 <?xml version="1.0"?>
 <robot xmlns:xacro="http://ros.org/wiki/xacro">
-    <xacro:property name="mesh_root" value="file://$(find urdf_visualize)/meshes"/>
+    <xacro:property name="mesh_root" value="file://$(find sambot_description)/meshes"/>
     <!-- MAIN LINK NAMES -->
     <xacro:property name="base_link_name" value="base_link"/>
@@ -45,4 +45,5 @@
     <xacro:property name="cabin_base_material" value="0.2314 0.3804 0.7059 1.0"/>
     <xacro:property name="cabin_base_inertial" value="3175.1655302028038932 -269.97312494382822479 167.61780128589879268 2627.6328649732372469 -193.85494965010886403 3742.616047274826542"/>
+    <!-- TURRET PARAMS -->
     <xacro:property name="turret_base_mesh" value="${mesh_root}/compact_excavator_frame_body.stl"/>
     <xacro:property name="turret_base_origin" value="0 0 0"/>
@@ -53,4 +54,5 @@
     <xacro:property name="turret_base_material" value="0.9176 0.9176 0.9176 1.0"/>
     <xacro:property name="turret_base_inertial" value="103.54309263053609413 2.8689912175751035583 -0.26918599165092144121 71.550382439979060223 -8.7881744003938315757 164.71779214088334697"/>
+    <!-- LEFT SPINNING (BACK) WHEEL -->
     <xacro:property name="left_spinning_wheel_link_mesh" value="${mesh_root}/compact_excavator_main_drive_wheel.stl"/>
     <xacro:property name="left_spinning_wheel_link_origin" value="0 -2.0816681711721685133e-17 -0.015000000000000124345"/>
@@ -61,4 +63,5 @@
     <xacro:property name="left_spinning_wheel_link_mass" value="35.986291345795820007"/>
     <xacro:property name="left_spinning_wheel_link_inertial" value="0.20071737580058110484 2.1151248144254331483e-17 7.9696042408110000254e-05 0.20066206838835709547 2.9623558171777900037e-16 0.29333573070696433716"/>
+    <!-- RIGHT SPINNING (BACK) WHEEL -->
     <xacro:property name="right_spinning_wheel_link_mesh" value="${mesh_root}/compact_excavator_main_drive_wheel.stl"/>
     <xacro:property name="right_spinning_wheel_link_origin" value="-6.9388939039072283776e-18 0 -0.015000000000000013323"/>
@@ -69,4 +72,5 @@
     <xacro:property name="right_spinning_wheel_link_mass" value="35.986291345795820007"/>
     <xacro:property name="right_spinning_wheel_link_inertial" value="0.20071737580058127137 6.1250580134766935832e-18 7.9696042408110027359e-05 0.20066206838835703996 2.9623106429686494369e-16 0.29333573070696433716"/>
+    <!-- LEFT FRONT WHEEL -->
     <xacro:property name="left_front_wheel_link_mesh" value="${mesh_root}/compact_excavator_front_wheel.stl"/>
     <xacro:property name="left_front_wheel_link_origin" value="1.1102230246251565404e-16 -1.1102230246251565404e-16 -0.032500000000000084377"/>
@@ -77,4 +81,5 @@
     <xacro:property name="left_front_wheel_link_mass" value="17.64673591392957519"/>
     <xacro:property name="left_front_wheel_link_inertial" value="0.153078316536178205 1.0629206596102168903e-17 2.6922495826861160064e-17 0.15307831653617814949 6.9747558075870228735e-33 0.29963755764746907717"/>
+    <!-- RIGHT FRONT WHEEL -->
     <xacro:property name="right_front_wheel_link_mesh" value="${mesh_root}/compact_excavator_front_wheel.stl"/>
     <xacro:property name="right_front_wheel_link_origin" value="-2.7755575615628913511e-17 0 -0.032500000000000084377"/>
@@ -85,4 +90,5 @@
     <xacro:property name="right_front_wheel_link_mass" value="17.64673591392957519"/>
     <xacro:property name="right_front_wheel_link_inertial" value="0.153078316536178205 -1.0629206596102168903e-17 2.6922495826861160064e-17 0.15307831653617814949 6.9747558075870228735e-33 0.29963755764746907717"/>
+    <!-- PLOW -->
     <xacro:property name="push_blade_base_mesh" value="${mesh_root}/push_blade_bucket.stl"/>
     <xacro:property name="push_blade_base_origin" value="-0.021564399534920564161 1.0799900599760599018 -0.25500000000000000444"/>
@@ -93,4 +99,5 @@
     <xacro:property name="push_blade_base_mass" value="147.01808168083425699"/>
     <xacro:property name="push_blade_base_inertial" value="31.881096131626421197 0.91247385061899932701 -1.6212090668492922982e-05 21.196220352263214437 4.9900082202379639952e-06 13.169227707961496776"/>
+    <!-- SWING -->
     <xacro:property name="swing_base_mesh" value="${mesh_root}/part01_pin_1.stl"/>
     <xacro:property name="swing_base_origin" value="2.7755575615628913511e-17 0.074999999999999955591 -0.14999999999999996669"/>
@@ -101,4 +108,5 @@
     <xacro:property name="swing_base_mass" value="98.140190062279060612"/>
     <xacro:property name="swing_base_inertial" value="2.6085778666185075458 0.040227300901953748358 0.42136783119553594679 3.1665232143977135593 -0.15916376835413623136 1.7889951810686841593"/>
+    <!-- BOOM -->
     <xacro:property name="boom_base_mesh" value="${mesh_root}/part02.stl"/>
     <xacro:property name="boom_base_origin" value="0 -1.1102230246251565404e-16 -0.079999999999999987788"/>
@@ -109,4 +117,5 @@
     <xacro:property name="boom_base_mass" value="694.17793513858055121"/>
     <xacro:property name="boom_base_inertial" value="242.81245205849677404 71.370938403077758494 0.0065905643878567711502 49.641340591529456105 -0.034260052091464154866 289.83702909122945357"/>
+    <!-- ARM -->
     <xacro:property name="arm_base_mesh" value="${mesh_root}/part03.stl"/>
     <xacro:property name="arm_base_origin" value="0 -2.2204460492503130808e-16 -0.054999999999999882316"/>
@@ -117,4 +126,5 @@
     <xacro:property name="arm_base_mass" value="265.34907807560875881"/>
     <xacro:property name="arm_base_inertial" value="57.599134249663784146 0.078442580554215754485 0.0049826290162324230956 1.8968981412117758012 0.02459901605653430981 58.868680211308259231"/>
+    <!-- BUCKET(S) -->
     <xacro:property name="bucket_mesh1" value="${mesh_root}/part04.stl"/>
     <xacro:property name="bucket_mesh1_origin" value="0.060000000000000053291 0.14000000000000012434 0.054999999999999993339"/>
@@ -133,8 +143,10 @@
     <xacro:property name="bucket_base_mass" value="132.70765933863819441"/>
     <xacro:property name="bucket_base_inertial" value="14.03567187790122972 -1.6652440163767181502 0.0020270508814650067472 6.8549730106956987541 0.0040437120644442776929 11.610921270718170817"/>
+    <!-- SKID WHEELS FOR DIFF DRIVE -->
     <xacro:property name="rubber_density" value="1100"/>
     <xacro:property name="wheel_radius" value="0.25"/>
     <xacro:property name="wheel_length" value="0.2"/>
     <xacro:macro name="skid_wheel" params="wheel_name mu1 mu2">
+        <!-- MULTIPLIED BY 100 TO ANCHOR -->
         <xacro:property name="wheel_mass" value="${100*3.1415*(wheel_radius**2)*wheel_length*rubber_density}"/>
         <xacro:property name="wheel_ixx" value="${(1/12)*wheel_mass*(3*wheel_radius**2 + wheel_length**2)}"/>

File: sambot_description/urdf/velocity/dynamics.xacro (robot description, xacro)
@@ -2,16 +2,5 @@
 <robot xmlns:xacro="http://ros.org/wiki/xacro">
     <xacro:include filename="$(find sambot_description)/urdf/params.xacro"/>
-    <xacro:macro name="gazebo_joint_dynamics" params="joint_name stiffness damping">
-        <gazebo reference="${joint_name}">
-            <stiffness>${stiffness}</stiffness>
-            <damping>${damping}</damping>
-            <!-- <pid>
-                <p>1</p>
-                <i>0</i>
-                <d>0</d>
-            </pid> -->
-            <dynamics damping="5000" friction="0.2"/>
-        </gazebo>
-    </xacro:macro>
+    <!-- EFFORT BASED JOINTS -->
     <xacro:macro name="gazebo_ros2_control_joints_effort" params="name effort_lim">
         <joint name="${name}">
@@ -26,4 +15,5 @@
         </joint>
     </xacro:macro>
+    <!-- VELOCITY BASED JOINTS -->
     <xacro:macro name="gazebo_ros2_control_joints_velocity" params="name velocity_lim">
         <joint name="${name}">
@@ -38,4 +28,5 @@
         </joint>
     </xacro:macro>
+    <!-- POSITION BASED JOINTS -->
     <xacro:macro name="gazebo_ros2_control_joints_position" params="name position_lim">
         <joint name="${name}">
@@ -49,4 +40,5 @@
         </joint>
     </xacro:macro>
+    <!-- TRANSMISSIONS FOR CONTROL (REQUIRED FOR ALL INTERFACES VIA ros2_control) -->
     <xacro:macro name="simple_transmission" params="name">
         <transmission name="${name}_trans">
@@ -61,14 +53,5 @@
         </transmission>
     </xacro:macro>
-    <xacro:gazebo_joint_dynamics joint_name="${excavator_slew_joint_name}" stiffness="30000" damping="5"/>
-    <xacro:gazebo_joint_dynamics joint_name="${plow_to_base_joint_name}" stiffness="30000" damping="5"/>
-    <xacro:gazebo_joint_dynamics joint_name="${arm_to_bucket_joint_name}" stiffness="30000" damping="5"/>
-    <xacro:gazebo_joint_dynamics joint_name="${boom_to_arm_joint_name}" stiffness="30000" damping="5"/>
-    <xacro:gazebo_joint_dynamics joint_name="${swing_to_boom_joint_name}" stiffness="30000" damping="5"/>
-    <xacro:gazebo_joint_dynamics joint_name="${cabin_to_swing_joint_name}" stiffness="30000" damping="5"/>
-    <xacro:gazebo_joint_dynamics joint_name="${left_spin_to_skid_joint_name}" stiffness="30000" damping="5"/>
-    <xacro:gazebo_joint_dynamics joint_name="${left_free_to_skid_joint_name}" stiffness="30000" damping="5"/>
-    <xacro:gazebo_joint_dynamics joint_name="${right_spin_to_skid_joint_name}" stiffness="30000" damping="5"/>
-    <xacro:gazebo_joint_dynamics joint_name="${right_free_to_skid_joint_name}" stiffness="30000" damping="5"/>
+    <!-- INSTANTIATE TRANSMISSIONS -->
     <xacro:simple_transmission name="${excavator_slew_joint_name}"/>
     <xacro:simple_transmission name="${plow_to_base_joint_name}"/>
@@ -77,4 +60,5 @@
     <xacro:simple_transmission name="${swing_to_boom_joint_name}"/>
     <xacro:simple_transmission name="${cabin_to_swing_joint_name}"/>
+    <!-- MAIN DYNAMICS -->
     <xacro:macro name="dynamics_plugins">
         <ros2_control name="GazeboSystem" type="system">

File: sambot_description/urdf/velocity/robot.xacro (robot description, xacro)
@@ -1,7 +1,9 @@
 <?xml version="1.0"?>
+<!-- BASE ROBOT XACRO -->
 <robot xmlns:xacro="http://www.ros.org/wiki/xacro" name="excavator">
+    <!-- EXCAVATOR SPECIFIC CONSTANTS -->
     <xacro:include filename="$(find sambot_description)/urdf/params.xacro" />
-    <xacro:include filename="$(find sambot_description)/urdf/joints.xacro" />
-    <xacro:include filename="$(find sambot_description)/urdf/velocity/dynamics.xacro" />
+    <!-- JOINTS AND THEIR DYNAMICS -->
+    <xacro:include filename="$(find sambot_description)/urdf/velocity/joints.xacro" />
     <link name="base_link"/>
     <link name="cabin_base">
@@ -354,4 +356,5 @@
         </collision>
     </link>
+    <!-- SKID WHEELS FOR SKID-STEER CONTROL -->
     <xacro:skid_wheel wheel_name="${left_skid_wheel_spinning_link_name}" mu1="1" mu2="1"/>
     <xacro:skid_wheel wheel_name="${left_skid_wheel_free_link_name}" mu1="1" mu2="1"/>
