Commit message: changed names to match params

File: sambot_description/urdf/dynamics.xacro (robot description, xacro)
@@ -1,4 +1,5 @@
 <?xml version="1.0"?>
 <robot xmlns:xacro="http://ros.org/wiki/xacro">
+    <xacro:include filename="$(find sambot_description)/urdf/params.xacro"/>
     <xacro:macro name="gazebo_joint_dynamics" params="joint_name stiffness damping">
         <gazebo reference="${joint_name}">
@@ -30,20 +31,20 @@
         </transmission>
     </xacro:macro>
-    <xacro:gazebo_joint_dynamics joint_name="excavator_slew" stiffness="1000" damping="0.1"/>
-    <xacro:gazebo_joint_dynamics joint_name="plow_to_base" stiffness="1000" damping="0.1"/>
-    <xacro:gazebo_joint_dynamics joint_name="arm_to_bucket" stiffness="1000" damping="0.1"/>
-    <xacro:gazebo_joint_dynamics joint_name="boom_to_arm" stiffness="1000" damping="0.1"/>
-    <xacro:gazebo_joint_dynamics joint_name="swing_to_boom" stiffness="1000" damping="0.1"/>
-    <xacro:gazebo_joint_dynamics joint_name="cabin_to_swing" stiffness="1000" damping="0.1"/>
-    <xacro:gazebo_joint_dynamics joint_name="left_spin_to_skid" stiffness="1000" damping="0.1"/>
-    <xacro:gazebo_joint_dynamics joint_name="left_free_to_skid" stiffness="1000" damping="0.1"/>
-    <xacro:gazebo_joint_dynamics joint_name="right_spin_to_skid" stiffness="1000" damping="0.1"/>
-    <xacro:gazebo_joint_dynamics joint_name="right_free_to_skid" stiffness="1000" damping="0.1"/>
-    <xacro:simple_transmission name="excavator_slew"/>
-    <xacro:simple_transmission name="plow_to_base"/>
-    <xacro:simple_transmission name="arm_to_bucket"/>
-    <xacro:simple_transmission name="boom_to_arm"/>
-    <xacro:simple_transmission name="swing_to_boom"/>
-    <xacro:simple_transmission name="cabin_to_swing"/>
+    <xacro:gazebo_joint_dynamics joint_name="${excavator_slew_joint_name}" stiffness="0" damping="5"/>
+    <xacro:gazebo_joint_dynamics joint_name="${plow_to_base_joint_name}" stiffness="0" damping="0.1"/>
+    <xacro:gazebo_joint_dynamics joint_name="${arm_to_bucket_joint_name}" stiffness="0" damping="0.1"/>
+    <xacro:gazebo_joint_dynamics joint_name="${boom_to_arm_joint_name}" stiffness="0" damping="0.1"/>
+    <xacro:gazebo_joint_dynamics joint_name="${swing_to_boom_joint_name}" stiffness="0" damping="0.1"/>
+    <xacro:gazebo_joint_dynamics joint_name="${cabin_to_swing_joint_name}" stiffness="0" damping="0.1"/>
+    <xacro:gazebo_joint_dynamics joint_name="${left_spin_to_skid_joint_name}" stiffness="0" damping="0.1"/>
+    <xacro:gazebo_joint_dynamics joint_name="${left_free_to_skid_joint_name}" stiffness="0" damping="0.1"/>
+    <xacro:gazebo_joint_dynamics joint_name="${right_spin_to_skid_joint_name}" stiffness="0" damping="0.1"/>
+    <xacro:gazebo_joint_dynamics joint_name="${right_free_to_skid_joint_name}" stiffness="0" damping="0.1"/>
+    <xacro:simple_transmission name="${excavator_slew_joint_name}"/>
+    <xacro:simple_transmission name="${plow_to_base_joint_name}"/>
+    <xacro:simple_transmission name="${arm_to_bucket_joint_name}"/>
+    <xacro:simple_transmission name="${boom_to_arm_joint_name}"/>
+    <xacro:simple_transmission name="${swing_to_boom_joint_name}"/>
+    <xacro:simple_transmission name="${cabin_to_swing_joint_name}"/>
     <xacro:macro name="dynamics_plugins">
         <ros2_control name="GazeboSystem" type="system">
@@ -51,10 +52,10 @@
                 <plugin>gazebo_ros2_control/GazeboSystem</plugin>
             </hardware>
-            <xacro:gazebo_ros2_control_joints name="excavator_slew" effort_lim="10000"/>
-            <xacro:gazebo_ros2_control_joints name="plow_to_base"  effort_lim="10000"/>
-            <xacro:gazebo_ros2_control_joints name="arm_to_bucket"  effort_lim="10000"/>
-            <xacro:gazebo_ros2_control_joints name="boom_to_arm"  effort_lim="10000"/>
-            <xacro:gazebo_ros2_control_joints name="swing_to_boom"  effort_lim="10000"/>
-            <xacro:gazebo_ros2_control_joints name="cabin_to_swing"  effort_lim="10000"/>
+            <xacro:gazebo_ros2_control_joints name="${excavator_slew_joint_name}" effort_lim="10000"/>
+            <xacro:gazebo_ros2_control_joints name="${plow_to_base_joint_name}"  effort_lim="10000"/>
+            <xacro:gazebo_ros2_control_joints name="${arm_to_bucket_joint_name}"  effort_lim="10000"/>
+            <xacro:gazebo_ros2_control_joints name="${boom_to_arm_joint_name}"  effort_lim="10000"/>
+            <xacro:gazebo_ros2_control_joints name="${swing_to_boom_joint_name}"  effort_lim="10000"/>
+            <xacro:gazebo_ros2_control_joints name="${cabin_to_swing_joint_name}"  effort_lim="10000"/>
         </ros2_control>
         <gazebo>
@@ -66,13 +67,13 @@
             <plugin name="two_wheeled_robot_diff_drive" filename="libgazebo_ros_diff_drive.so">
                 <num_wheel_pairs>2</num_wheel_pairs>
-                <left_joint>left_spinning_wheel</left_joint>
-                <left_joint>left_passive_wheel</left_joint>
-                <right_joint>right_spinning_wheel</right_joint>
-                <right_joint>right_passive_wheel</right_joint>
+                <left_joint>${left_spinning_to_turret_joint_name}</left_joint>
+                <left_joint>${left_front_to_turret_joint_name}</left_joint>
+                <right_joint>${right_spinning_to_turret_joint_name}</right_joint>
+                <right_joint>${right_front_to_turret_joint_name}</right_joint>
                 <wheel_separation>1.75</wheel_separation>
                 <wheel_separation>1.75</wheel_separation>
                 <wheel_diameter>${wheel_radius*2}</wheel_diameter>
                 <wheel_diameter>${wheel_radius*2}</wheel_diameter>
-                <max_wheel_torque>1000</max_wheel_torque>
+                <max_wheel_torque>10000</max_wheel_torque>
                 <max_wheel_acceleration>1.0</max_wheel_acceleration>
                 <publish_odom>true</publish_odom>

File: sambot_description/urdf/joints.xacro (robot description, xacro)
@@ -1,93 +1,93 @@
 <?xml version="1.0"?>
 <robot xmlns:xacro="http://ros.org/wiki/xacro">
+    <xacro:include filename="$(find sambot_description)/urdf/params.xacro"/>
     <xacro:macro name="dynamics" params="dyn_damping dyn_friction">
             <dynamics damping="${dyn_damping}" friction="${dyn_friction}"/>
     </xacro:macro>
-    <joint name="left_spin_to_skid" type="fixed">
+    <joint name="${left_spin_to_skid_joint_name}" type="fixed">
         <origin xyz="0 0 -0.3" rpy="0 0 0"/>
-        <parent link="left_spinning_wheel_link"/>
-        <child link="left_skid_wheel_spinning"/>
+        <parent link="${left_spinning_wheel_link_name}"/>
+        <child link="${left_skid_wheel_spinning_link_name}"/>
         <axis xyz="0 0 1"/>
         <xacro:dynamics dyn_damping="0.1" dyn_friction="0.0"/>
     </joint>
-    <joint name="left_free_to_skid" type="fixed">
+    <joint name="${left_free_to_skid_joint_name}" type="fixed">
         <origin xyz="0 0 0.3" rpy="0 0 0"/>
-        <parent link="left_front_wheel_link"/>
-        <child link="left_skid_wheel_free"/>
+        <parent link="${left_front_wheel_link_name}"/>
+        <child link="${left_skid_wheel_free_link_name}"/>
         <axis xyz="0 0 1"/>
         <xacro:dynamics dyn_damping="0.1" dyn_friction="0.0"/>
     </joint>
-    <joint name="right_spin_to_skid" type="fixed">
+    <joint name="${right_spin_to_skid_joint_name}" type="fixed">
         <origin xyz="0 0 -0.3" rpy="0 0 0"/>
-        <parent link="right_spinning_wheel_link"/>
-        <child link="right_skid_wheel_spinning"/>
+        <parent link="${right_spinning_wheel_link_name}"/>
+        <child link="${right_skid_wheel_spinning_link_name}"/>
         <axis xyz="0 0 1"/>
         <xacro:dynamics dyn_damping="0.1" dyn_friction="0.0"/>
     </joint>
-    <joint name="right_free_to_skid" type="fixed">
+    <joint name="${right_free_to_skid_joint_name}" type="fixed">
         <origin xyz="0 0 -0.3" rpy="0 0 0"/>
-        <parent link="right_front_wheel_link"/>
-        <child link="right_skid_wheel_free"/>
+        <parent link="${right_front_wheel_link_name}"/>
+        <child link="${right_skid_wheel_free_link_name}"/>
+        <axis xyz="0 0 1"/>
+        <xacro:dynamics dyn_damping="0.1" dyn_friction="0.0"/>
+    </joint>
+    <joint name="${base_to_turret_joint_name}" type="fixed">
+        <origin xyz="0 0 0.55" rpy="0 0 0" />
+        <parent link="${base_link_name}" />
+        <child link="${turret_link_name}" />
+        <axis xyz="0 0 1"/>
+    </joint>
+    <joint name="${left_spinning_to_turret_joint_name}" type="continuous">
+        <origin xyz="-0.5739999999999999547 -0.80000000000000015543 -0.2750000000000000222" rpy="1.570796326794896558 -0.3547477759675310427 1.5707963267948976682" />
+        <parent link="${turret_link_name}" />
+        <child link="${left_spinning_wheel_link_name}" />
+        <axis xyz="0 0 1"/>
+        <limit effort="10000" velocity="5" />
+        <xacro:dynamics dyn_damping="0.1" dyn_friction="0.0"/>
+    </joint>
+    <joint name="${right_spinning_to_turret_joint_name}" type="continuous">
+        <origin xyz="0.5739999999999999547 -0.80000000000000004441 -0.2750000000000000222" rpy="1.570796326794896558 -1.2984776443375001254 -1.5707963267948972241" />
+        <parent link="${turret_link_name}" />
+        <child link="${right_spinning_wheel_link_name}" />
+        <axis xyz="0 0 1"/>
+        <limit effort="10000" velocity="5" />
+        <xacro:dynamics dyn_damping="0.1" dyn_friction="0.0"/>
+    </joint>
+    <joint name="${left_front_to_turret_joint_name}" type="continuous">
+        <origin xyz="-0.61299999999999998934 0.80000000000000026645 -0.2750000000000000222" rpy="1.570796326794896558 -1.0222876983448163646 -1.5707963267948941155" />
+        <parent link="${turret_link_name}" />
+        <child link="${left_front_wheel_link_name}" />
+        <axis xyz="0 0 1"/>
+        <limit effort="10000" velocity="5" />
+        <xacro:dynamics dyn_damping="0.1" dyn_friction="0.0"/>
+    </joint>
+    <joint name="${right_front_to_turret_joint_name}" type="continuous">
+        <origin xyz="0.54800000000000004263 0.80000000000000015543 -0.27499999999999996669" rpy="1.57079632679489678 -1.1102232252180887662e-16 -1.5707963267948976682" />
+        <parent link="${turret_link_name}" />
+        <child link="${right_front_wheel_link_name}" />
+        <axis xyz="0 0 1"/>
+        <limit effort="10000" velocity="5" />
+        <xacro:dynamics dyn_damping="0.1" dyn_friction="0.0"/>
+    </joint>
+    <joint name="${plow_to_base_joint_name}" type="revolute">
+        <origin xyz="-0.25500000000000005995 0.4880000000000002669 -0.20500000000000001554" rpy="1.570796326794896558 -1.3195606112546109934 -1.57079632679489678" />
+        <parent link="${turret_link_name}" />
+        <child link="${plow_link_name}" />
+        <axis xyz="0 0 1"/>
+        <limit effort="10000" velocity="5" lower="0.2" upper="0" />
+        <xacro:dynamics dyn_damping="0.1" dyn_friction="0.0"/>
+    </joint>
+    <joint name="${excavator_slew_joint_name}" type="continuous">
+        <origin xyz="0 0 0.1" rpy="-5.5511151231419568159e-17 -1.1102230246202266528e-16 -3.1415" />
+        <parent link="${turret_link_name}" />
+        <child link="${cabin_link_name}" />
         <axis xyz="0 0 1"/>
         <limit effort="10000" velocity="5"/>
         <xacro:dynamics dyn_damping="0.1" dyn_friction="0.0"/>
     </joint>
-    <joint name="base_to_turret" type="fixed">
-        <origin xyz="0 0 0.55" rpy="0 0 0" />
-        <parent link="base_link" />
-        <child link="turret_base" />
-        <axis xyz="0 0 1"/>
-    </joint>
-    <joint name="left_spinning_wheel" type="continuous">
-        <origin xyz="-0.5739999999999999547 -0.80000000000000015543 -0.2750000000000000222" rpy="1.570796326794896558 -0.3547477759675310427 1.5707963267948976682" />
-        <parent link="turret_base" />
-        <child link="left_spinning_wheel_link" />
-        <axis xyz="0 0 1"/>
-        <limit effort="10000" velocity="5" />
-        <xacro:dynamics dyn_damping="0.1" dyn_friction="0.0"/>
-    </joint>
-    <joint name="right_spinning_wheel" type="continuous">
-        <origin xyz="0.5739999999999999547 -0.80000000000000004441 -0.2750000000000000222" rpy="1.570796326794896558 -1.2984776443375001254 -1.5707963267948972241" />
-        <parent link="turret_base" />
-        <child link="right_spinning_wheel_link" />
-        <axis xyz="0 0 1"/>
-        <limit effort="10000" velocity="5" />
-        <xacro:dynamics dyn_damping="0.1" dyn_friction="0.0"/>
-    </joint>
-    <joint name="left_passive_wheel" type="continuous">
-        <origin xyz="-0.61299999999999998934 0.80000000000000026645 -0.2750000000000000222" rpy="1.570796326794896558 -1.0222876983448163646 -1.5707963267948941155" />
-        <parent link="turret_base" />
-        <child link="left_front_wheel_link" />
-        <axis xyz="0 0 1"/>
-        <limit effort="10000" velocity="5" />
-        <xacro:dynamics dyn_damping="0.1" dyn_friction="0.0"/>
-    </joint>
-    <joint name="right_passive_wheel" type="continuous">
-        <origin xyz="0.54800000000000004263 0.80000000000000015543 -0.27499999999999996669" rpy="1.57079632679489678 -1.1102232252180887662e-16 -1.5707963267948976682" />
-        <parent link="turret_base" />
-        <child link="right_front_wheel_link" />
-        <axis xyz="0 0 1"/>
-        <limit effort="10000" velocity="5" />
-        <xacro:dynamics dyn_damping="0.1" dyn_friction="0.0"/>
-    </joint>
-    <joint name="plow_to_base" type="revolute">
-        <origin xyz="-0.25500000000000005995 0.4880000000000002669 -0.20500000000000001554" rpy="1.570796326794896558 -1.3195606112546109934 -1.57079632679489678" />
-        <parent link="turret_base" />
-        <child link="push_blade_base" />
-        <axis xyz="0 0 1"/>
-        <limit effort="10000" velocity="5" lower="0.2" upper="0" />
-        <xacro:dynamics dyn_damping="0.1" dyn_friction="0.0"/>
-    </joint>
-    <joint name="excavator_slew" type="continuous">
-        <origin xyz="0 0 0.1" rpy="-5.5511151231419568159e-17 -1.1102230246202266528e-16 -3.1415" />
-        <parent link="turret_base" />
-        <child link="cabin_base" />
-        <axis xyz="0 0 1"/>
-        <limit effort="10000" velocity="5"/>
-        <xacro:dynamics dyn_damping="0.1" dyn_friction="0.0"/>
-    </joint>
-    <joint name="arm_to_bucket" type="revolute">
+    <joint name="${arm_to_bucket_joint_name}" type="revolute">
         <origin xyz="0.12000000000000410338 -1.5403327562575612752 9.4368957093138305936e-16" rpy="3.1415926535897917837 1.8859935444767496044e-16 -1.5963552846072552871" />
-        <parent link="arm_base" />
+        <parent link="${arm_link_name}" />
         <child link="bucket_base" />
         <axis xyz="0 0 1"/>
@@ -95,24 +95,24 @@
         <xacro:dynamics dyn_damping="0.1" dyn_friction="0.0"/>
     </joint>
-    <joint name="boom_to_arm" type="revolute">
+    <joint name="${boom_to_arm_joint_name}" type="revolute">
         <origin xyz="-0.84000000000000030198 2.3549999999999999822 -0.13500000000000003664" rpy="3.1415926535897922278 6.9325343981756730312e-15 2.5555644018935783635" />
-        <parent link="boom_base" />
-        <child link="arm_base" />
+        <parent link="${boom_link_name}" />
+        <child link="${arm_link_name}" />
         <axis xyz="0 0 1"/>
         <limit effort="10000" velocity="5" lower="-0.5" upper="1.57"/>
         <xacro:dynamics dyn_damping="0.1" dyn_friction="0.0"/>
     </joint>
-    <joint name="swing_to_boom" type="revolute">
+    <joint name="${swing_to_boom_joint_name}" type="revolute">
         <origin xyz="0.079999999999996157518 0.074999999999997291056 -0.1500000000000039635" rpy="-1.570796326794896558 0.39285813115170314935 -1.5707963267949009989" />
-        <parent link="swing_base" />
-        <child link="boom_base" />
+        <parent link="${swing_link_name}" />
+        <child link="${boom_link_name}" />
         <axis xyz="0 0 1"/>
-        <limit effort="10000" velocity="5" lower="-0.4" upper="0.4" />
+        <limit effort="10000" velocity="5" lower="-0.1" upper="0.1" />
         <xacro:dynamics dyn_damping="0.1" dyn_friction="0.0"/>
     </joint>
-    <joint name="cabin_to_swing" type="revolute">
+    <joint name="${cabin_to_swing_joint_name}" type="revolute">
         <origin xyz="-0.040707723917193447405 -0.80673603465099630316 0.38039999999999996039" rpy="3.141592653589793116 4.8797124238540929311e-17 0.21446312817660284633" />
-        <parent link="cabin_base" />
-        <child link="swing_base" />
+        <parent link="${cabin_link_name}" />
+        <child link="${swing_link_name}" />
         <axis xyz="0 0 1"/>
         <limit effort="10000" velocity="5" lower="-1" upper="1.57" />

File: sambot_description/urdf/params.xacro (robot description, xacro)
@@ -2,4 +2,39 @@
 <robot xmlns:xacro="http://ros.org/wiki/xacro">
     <xacro:property name="mesh_root" value="file://$(find urdf_visualize)/meshes"/>
+    <!-- MAIN LINK NAMES -->
+    <xacro:property name="base_link_name" value="base_link"/>
+    <xacro:property name="cabin_link_name" value="cabin_base"/>
+    <xacro:property name="turret_link_name" value="turret_base"/>
+    <xacro:property name="plow_link_name" value="push_blade_base"/>
+    <xacro:property name="swing_link_name" value="swing_base"/>
+    <xacro:property name="boom_link_name" value="boom_base"/>
+    <xacro:property name="arm_link_name" value="arm_base"/>
+    <xacro:property name="bucket_link_name" value="bucket_base"/>
+    <!-- WHEEL LINKS -->
+    <xacro:property name="left_spinning_wheel_link_name" value="left_spinning_wheel_link"/>
+    <xacro:property name="right_spinning_wheel_link_name" value="right_spinning_wheel_link"/>
+    <xacro:property name="left_front_wheel_link_name" value="left_front_wheel_link"/>
+    <xacro:property name="right_front_wheel_link_name" value="right_front_wheel_link"/>
+    <xacro:property name="left_skid_wheel_spinning_link_name" value="left_skid_wheel_spinning"/>
+    <xacro:property name="left_skid_wheel_free_link_name" value="left_skid_wheel_free"/>
+    <xacro:property name="right_skid_wheel_spinning_link_name" value="right_skid_wheel_spinning"/>
+    <xacro:property name="right_skid_wheel_free_link_name" value="right_skid_wheel_free"/>
+    <!-- JOINT NAMES -->
+    <xacro:property name="base_to_turret_joint_name" value="base_to_turret"/>
+    <xacro:property name="left_spinning_to_turret_joint_name" value="left_spinning_to_turret"/>
+    <xacro:property name="left_front_to_turret_joint_name" value="left_front_to_turret"/>
+    <xacro:property name="right_spinning_to_turret_joint_name" value="right_spinning_to_turret"/>
+    <xacro:property name="right_front_to_turret_joint_name" value="right_front_to_turret"/>
+    <xacro:property name="plow_to_base_joint_name" value="plow_to_base"/>
+    <xacro:property name="swing_to_boom_joint_name" value="swing_to_boom"/>
+    <xacro:property name="boom_to_arm_joint_name" value="boom_to_arm"/>
+    <xacro:property name="arm_to_bucket_joint_name" value="arm_to_bucket"/>
+    <xacro:property name="cabin_to_swing_joint_name" value="cabin_to_swing"/>
+    <xacro:property name="excavator_slew_joint_name" value="excavator_slew"/>
+    <xacro:property name="left_spin_to_skid_joint_name" value="left_spin_to_skid"/>
+    <xacro:property name="left_free_to_skid_joint_name" value="left_free_to_skid"/>
+    <xacro:property name="right_spin_to_skid_joint_name" value="right_spin_to_skid"/>
+    <xacro:property name="right_free_to_skid_joint_name" value="right_free_to_skid"/>
+    <!-- CABIN LINK PARAMS -->
     <xacro:property name="cabin_base_mesh" value="${mesh_root}/compact_excavator_cabin_body.stl"/>
     <xacro:property name="cabin_base_origin" value="0.1592 -0.2513 0.2814"/>
@@ -82,5 +117,4 @@
     <xacro:property name="arm_base_mass" value="265.34907807560875881"/>
     <xacro:property name="arm_base_inertial" value="57.599134249663784146 0.078442580554215754485 0.0049826290162324230956 1.8968981412117758012 0.02459901605653430981 58.868680211308259231"/>
-    <xacro:property name="bucket_link_name" value="bucket_base"/>
     <xacro:property name="bucket_mesh1" value="${mesh_root}/part04.stl"/>
     <xacro:property name="bucket_mesh1_origin" value="0.060000000000000053291 0.14000000000000012434 0.054999999999999993339"/>

File: sambot_description/urdf/robot.xacro (robot description, xacro)
@@ -354,8 +354,8 @@
         </collision>
     </link>
-    <xacro:skid_wheel wheel_name="left_skid_wheel_spinning" mu1="1" mu2="1"/>
-    <xacro:skid_wheel wheel_name="left_skid_wheel_free" mu1="1" mu2="1"/>
-    <xacro:skid_wheel wheel_name="right_skid_wheel_spinning" mu1="1" mu2="1"/>
-    <xacro:skid_wheel wheel_name="right_skid_wheel_free" mu1="1" mu2="1"/>
+    <xacro:skid_wheel wheel_name="${left_skid_wheel_spinning_link_name}" mu1="1" mu2="1"/>
+    <xacro:skid_wheel wheel_name="${left_skid_wheel_free_link_name}" mu1="1" mu2="1"/>
+    <xacro:skid_wheel wheel_name="${right_skid_wheel_spinning_link_name}" mu1="1" mu2="1"/>
+    <xacro:skid_wheel wheel_name="${right_skid_wheel_free_link_name}" mu1="1" mu2="1"/>
     <xacro:dynamics_plugins/>
 </robot>
