Commit message: boom works for 15k effort

File: sambot_description/urdf/dynamics.xacro (robot description, xacro)
@@ -6,11 +6,28 @@
             <stiffness>${stiffness}</stiffness>
             <damping>${damping}</damping>
+            <pid>
+                <p>10</p>
+                <i>0</i>
+                <d>0.01</d>
+            </pid>
+            <dynamics damping="0.1" friction="0.2"/>
         </gazebo>
     </xacro:macro>
-    <xacro:macro name="gazebo_ros2_control_joints" params="name effort_lim">
+    <xacro:macro name="gazebo_ros2_control_joints_effort" params="name effort_lim">
         <joint name="${name}">
             <command_interface name="effort">
                 <param name="min">${-effort_lim}</param>
                 <param name="max">${effort_lim}</param>
+            </command_interface>
+            <state_interface name="position"/>
+            <state_interface name="velocity"/>
+            <state_interface name="effort"/>
+        </joint>
+    </xacro:macro>
+    <xacro:macro name="gazebo_ros2_control_joints_velocity" params="name velocity_lim">
+        <joint name="${name}">
+            <command_interface name="velocity">
+                <param name="min">${-velocity_lim}</param>
+                <param name="max">${velocity_lim}</param>
             </command_interface>
             <state_interface name="position"/>
@@ -31,14 +48,14 @@
         </transmission>
     </xacro:macro>
-    <xacro:gazebo_joint_dynamics joint_name="${excavator_slew_joint_name}" stiffness="0" damping="5"/>
-    <xacro:gazebo_joint_dynamics joint_name="${plow_to_base_joint_name}" stiffness="0" damping="0.1"/>
-    <xacro:gazebo_joint_dynamics joint_name="${arm_to_bucket_joint_name}" stiffness="0" damping="0.1"/>
-    <xacro:gazebo_joint_dynamics joint_name="${boom_to_arm_joint_name}" stiffness="0" damping="0.1"/>
-    <xacro:gazebo_joint_dynamics joint_name="${swing_to_boom_joint_name}" stiffness="0" damping="0.1"/>
-    <xacro:gazebo_joint_dynamics joint_name="${cabin_to_swing_joint_name}" stiffness="0" damping="0.1"/>
-    <xacro:gazebo_joint_dynamics joint_name="${left_spin_to_skid_joint_name}" stiffness="0" damping="0.1"/>
-    <xacro:gazebo_joint_dynamics joint_name="${left_free_to_skid_joint_name}" stiffness="0" damping="0.1"/>
-    <xacro:gazebo_joint_dynamics joint_name="${right_spin_to_skid_joint_name}" stiffness="0" damping="0.1"/>
-    <xacro:gazebo_joint_dynamics joint_name="${right_free_to_skid_joint_name}" stiffness="0" damping="0.1"/>
+    <xacro:gazebo_joint_dynamics joint_name="${excavator_slew_joint_name}" stiffness="3000" damping="5"/>
+    <xacro:gazebo_joint_dynamics joint_name="${plow_to_base_joint_name}" stiffness="3000" damping="0.1"/>
+    <xacro:gazebo_joint_dynamics joint_name="${arm_to_bucket_joint_name}" stiffness="3000" damping="0.1"/>
+    <xacro:gazebo_joint_dynamics joint_name="${boom_to_arm_joint_name}" stiffness="3000" damping="0.1"/>
+    <xacro:gazebo_joint_dynamics joint_name="${swing_to_boom_joint_name}" stiffness="3000" damping="0.1"/>
+    <xacro:gazebo_joint_dynamics joint_name="${cabin_to_swing_joint_name}" stiffness="3000" damping="0.1"/>
+    <xacro:gazebo_joint_dynamics joint_name="${left_spin_to_skid_joint_name}" stiffness="3000" damping="0.1"/>
+    <xacro:gazebo_joint_dynamics joint_name="${left_free_to_skid_joint_name}" stiffness="3000" damping="0.1"/>
+    <xacro:gazebo_joint_dynamics joint_name="${right_spin_to_skid_joint_name}" stiffness="3000" damping="0.1"/>
+    <xacro:gazebo_joint_dynamics joint_name="${right_free_to_skid_joint_name}" stiffness="3000" damping="0.1"/>
     <xacro:simple_transmission name="${excavator_slew_joint_name}"/>
     <xacro:simple_transmission name="${plow_to_base_joint_name}"/>
@@ -52,10 +69,16 @@
                 <plugin>gazebo_ros2_control/GazeboSystem</plugin>
             </hardware>
-            <xacro:gazebo_ros2_control_joints name="${excavator_slew_joint_name}" effort_lim="10000"/>
-            <xacro:gazebo_ros2_control_joints name="${plow_to_base_joint_name}"  effort_lim="10000"/>
-            <xacro:gazebo_ros2_control_joints name="${arm_to_bucket_joint_name}"  effort_lim="10000"/>
-            <xacro:gazebo_ros2_control_joints name="${boom_to_arm_joint_name}"  effort_lim="10000"/>
-            <xacro:gazebo_ros2_control_joints name="${swing_to_boom_joint_name}"  effort_lim="10000"/>
-            <xacro:gazebo_ros2_control_joints name="${cabin_to_swing_joint_name}"  effort_lim="10000"/>
+            <xacro:gazebo_ros2_control_joints_effort name="${excavator_slew_joint_name}" effort_lim="100000"/>
+            <xacro:gazebo_ros2_control_joints_effort name="${plow_to_base_joint_name}"  effort_lim="100000"/>
+            <xacro:gazebo_ros2_control_joints_effort name="${arm_to_bucket_joint_name}"  effort_lim="100000"/>
+            <xacro:gazebo_ros2_control_joints_effort name="${boom_to_arm_joint_name}"  effort_lim="100000"/>
+            <xacro:gazebo_ros2_control_joints_effort name="${swing_to_boom_joint_name}"  effort_lim="100000"/>
+            <xacro:gazebo_ros2_control_joints_effort name="${cabin_to_swing_joint_name}"  effort_lim="100000"/>
+            <!-- <xacro:gazebo_ros2_control_joints_velocity name="${excavator_slew_joint_name}" velocity_lim="1.0"/>
+            <xacro:gazebo_ros2_control_joints_velocity name="${plow_to_base_joint_name}"  velocity_lim="1.0"/>
+            <xacro:gazebo_ros2_control_joints_velocity name="${arm_to_bucket_joint_name}"  velocity_lim="1.0"/>
+            <xacro:gazebo_ros2_control_joints_velocity name="${boom_to_arm_joint_name}"  velocity_lim="1.0"/>
+            <xacro:gazebo_ros2_control_joints_velocity name="${swing_to_boom_joint_name}"  velocity_lim="1.0"/>
+            <xacro:gazebo_ros2_control_joints_velocity name="${cabin_to_swing_joint_name}"  velocity_lim="1.0"/> -->
         </ros2_control>
         <gazebo>

File: sambot_description/urdf/joints.xacro (robot description, xacro)
@@ -3,5 +3,5 @@
     <xacro:include filename="$(find sambot_description)/urdf/params.xacro"/>
     <xacro:macro name="dynamics" params="dyn_damping dyn_friction">
-            <dynamics damping="${dyn_damping}" friction="${dyn_friction}"/>
+            <!-- <dynamics damping="${dyn_damping}" friction="${dyn_friction}"/> -->
     </xacro:macro>
     <joint name="${left_spin_to_skid_joint_name}" type="fixed">
@@ -10,5 +10,5 @@
         <child link="${left_skid_wheel_spinning_link_name}"/>
         <axis xyz="0 0 1"/>
-        <xacro:dynamics dyn_damping="0.1" dyn_friction="0.0"/>
+        <!-- <xacro:dynamics dyn_damping="0.1" dyn_friction="0.2"/> -->
     </joint>
     <joint name="${left_free_to_skid_joint_name}" type="fixed">
@@ -17,5 +17,5 @@
         <child link="${left_skid_wheel_free_link_name}"/>
         <axis xyz="0 0 1"/>
-        <xacro:dynamics dyn_damping="0.1" dyn_friction="0.0"/>
+        <!-- <xacro:dynamics dyn_damping="0.1" dyn_friction="0.2"/> -->
     </joint>
     <joint name="${right_spin_to_skid_joint_name}" type="fixed">
@@ -24,5 +24,5 @@
         <child link="${right_skid_wheel_spinning_link_name}"/>
         <axis xyz="0 0 1"/>
-        <xacro:dynamics dyn_damping="0.1" dyn_friction="0.0"/>
+        <!-- <xacro:dynamics dyn_damping="0.1" dyn_friction="0.2"/> -->
     </joint>
     <joint name="${right_free_to_skid_joint_name}" type="fixed">
@@ -31,5 +31,5 @@
         <child link="${right_skid_wheel_free_link_name}"/>
         <axis xyz="0 0 1"/>
-        <xacro:dynamics dyn_damping="0.1" dyn_friction="0.0"/>
+        <!-- <xacro:dynamics dyn_damping="0.1" dyn_friction="0.2"/> -->
     </joint>
     <joint name="${base_to_turret_joint_name}" type="fixed">
@@ -44,6 +44,6 @@
         <child link="${left_spinning_wheel_link_name}" />
         <axis xyz="0 0 1"/>
-        <limit effort="10000" velocity="5" />
-        <xacro:dynamics dyn_damping="0.1" dyn_friction="0.0"/>
+        <limit effort="20000" velocity="5" />
+        <!-- <xacro:dynamics dyn_damping="0.1" dyn_friction="0.2"/> -->
     </joint>
     <joint name="${right_spinning_to_turret_joint_name}" type="continuous">
@@ -52,6 +52,6 @@
         <child link="${right_spinning_wheel_link_name}" />
         <axis xyz="0 0 1"/>
-        <limit effort="10000" velocity="5" />
-        <xacro:dynamics dyn_damping="0.1" dyn_friction="0.0"/>
+        <limit effort="20000" velocity="5" />
+        <!-- <xacro:dynamics dyn_damping="0.1" dyn_friction="0.2"/> -->
     </joint>
     <joint name="${left_front_to_turret_joint_name}" type="continuous">
@@ -60,6 +60,6 @@
         <child link="${left_front_wheel_link_name}" />
         <axis xyz="0 0 1"/>
-        <limit effort="10000" velocity="5" />
-        <xacro:dynamics dyn_damping="0.1" dyn_friction="0.0"/>
+        <limit effort="20000" velocity="5" />
+        <!-- <xacro:dynamics dyn_damping="0.1" dyn_friction="0.2"/> -->
     </joint>
     <joint name="${right_front_to_turret_joint_name}" type="continuous">
@@ -68,6 +68,6 @@
         <child link="${right_front_wheel_link_name}" />
         <axis xyz="0 0 1"/>
-        <limit effort="10000" velocity="5" />
-        <xacro:dynamics dyn_damping="0.1" dyn_friction="0.0"/>
+        <limit effort="20000" velocity="5" />
+        <!-- <xacro:dynamics dyn_damping="0.1" dyn_friction="0.2"/> -->
     </joint>
     <joint name="${plow_to_base_joint_name}" type="revolute">
@@ -76,6 +76,6 @@
         <child link="${plow_link_name}" />
         <axis xyz="0 0 1"/>
-        <limit effort="10000" velocity="5" lower="0.2" upper="0" />
-        <xacro:dynamics dyn_damping="0.1" dyn_friction="0.0"/>
+        <limit effort="20000" velocity="5" lower="0.2" upper="0" />
+        <!-- <xacro:dynamics dyn_damping="0.1" dyn_friction="0.2"/> -->
     </joint>
     <joint name="${excavator_slew_joint_name}" type="continuous">
@@ -84,6 +84,6 @@
         <child link="${cabin_link_name}" />
         <axis xyz="0 0 1"/>
-        <limit effort="10000" velocity="5"/>
-        <xacro:dynamics dyn_damping="0.1" dyn_friction="0.0"/>
+        <limit effort="20000" velocity="5"/>
+        <!-- <xacro:dynamics dyn_damping="0.1" dyn_friction="0.2"/> -->
     </joint>
     <joint name="${arm_to_bucket_joint_name}" type="revolute">
@@ -92,6 +92,6 @@
         <child link="bucket_base" />
         <axis xyz="0 0 1"/>
-        <limit effort="10000" velocity="5" lower="-1.2217304763960306069" upper="0.87266462599716476678"/>
-        <xacro:dynamics dyn_damping="0.1" dyn_friction="0.0"/>
+        <limit effort="20000" velocity="5" lower="-1.2217304763960306069" upper="0.87266462599716476678"/>
+        <!-- <xacro:dynamics dyn_damping="0.1" dyn_friction="0.2"/> -->
     </joint>
     <joint name="${boom_to_arm_joint_name}" type="revolute">
@@ -100,6 +100,6 @@
         <child link="${arm_link_name}" />
         <axis xyz="0 0 1"/>
-        <limit effort="10000" velocity="5" lower="-0.5" upper="1.57"/>
-        <xacro:dynamics dyn_damping="0.1" dyn_friction="0.0"/>
+        <limit effort="20000" velocity="5" lower="-0.5" upper="1.57"/>
+        <!-- <xacro:dynamics dyn_damping="0.1" dyn_friction="0.2"/> -->
     </joint>
     <joint name="${swing_to_boom_joint_name}" type="revolute">
@@ -108,14 +108,14 @@
         <child link="${boom_link_name}" />
         <axis xyz="0 0 1"/>
-        <limit effort="10000" velocity="5" lower="-0.1" upper="0.1" />
-        <xacro:dynamics dyn_damping="0.1" dyn_friction="0.0"/>
+        <limit effort="20000" velocity="5" lower="-1" upper="1" />
+        <!-- <xacro:dynamics dyn_damping="0.1" dyn_friction="0.2"/> -->
     </joint>
     <joint name="${cabin_to_swing_joint_name}" type="revolute">
-        <origin xyz="-0.040707723917193447405 -0.80673603465099630316 0.38039999999999996039" rpy="3.141592653589793116 4.8797124238540929311e-17 0.21446312817660284633" />
+        <origin xyz="-0.040707723917193447405 -0.80673603465099630316 0.38039999999999996039" rpy="3.141592653589793116 4.8797124238540929311e-17 0" />
         <parent link="${cabin_link_name}" />
         <child link="${swing_link_name}" />
         <axis xyz="0 0 1"/>
-        <limit effort="10000" velocity="5" lower="-1" upper="1.57" />
-        <xacro:dynamics dyn_damping="0.1" dyn_friction="0.0"/>
+        <limit effort="20000" velocity="5" lower="-0.1" upper="0.1" />
+        <!-- <xacro:dynamics dyn_damping="0.1" dyn_friction="0.2"/> -->
     </joint>
 </robot>

Commit message: position control works

File: sambot_description/urdf/dynamics.xacro (robot description, xacro)
@@ -7,9 +7,9 @@
             <damping>${damping}</damping>
             <pid>
-                <p>10</p>
+                <p>3000000</p>
                 <i>0</i>
-                <d>0.01</d>
+                <d>0</d>
             </pid>
-            <dynamics damping="0.1" friction="0.2"/>
+            <!-- <dynamics damping="0.1" friction="0.2"/> -->
         </gazebo>
     </xacro:macro>
@@ -22,5 +22,5 @@
             <state_interface name="position"/>
             <state_interface name="velocity"/>
-            <state_interface name="effort"/>
+            <!-- <state_interface name="effort"/> -->
         </joint>
     </xacro:macro>
@@ -34,4 +34,15 @@
             <state_interface name="velocity"/>
             <state_interface name="effort"/>
+        </joint>
+    </xacro:macro>
+    <xacro:macro name="gazebo_ros2_control_joints_position" params="name position_lim">
+        <joint name="${name}">
+            <command_interface name="position">
+                <param name="min">${-position_lim}</param>
+                <param name="max">${position_lim}</param>
+            </command_interface>
+            <state_interface name="position"/>
+            <state_interface name="velocity"/>
+            <!-- <state_interface name="effort"/> -->
         </joint>
     </xacro:macro>
@@ -48,14 +59,14 @@
         </transmission>
     </xacro:macro>
-    <xacro:gazebo_joint_dynamics joint_name="${excavator_slew_joint_name}" stiffness="3000" damping="5"/>
-    <xacro:gazebo_joint_dynamics joint_name="${plow_to_base_joint_name}" stiffness="3000" damping="0.1"/>
-    <xacro:gazebo_joint_dynamics joint_name="${arm_to_bucket_joint_name}" stiffness="3000" damping="0.1"/>
-    <xacro:gazebo_joint_dynamics joint_name="${boom_to_arm_joint_name}" stiffness="3000" damping="0.1"/>
-    <xacro:gazebo_joint_dynamics joint_name="${swing_to_boom_joint_name}" stiffness="3000" damping="0.1"/>
-    <xacro:gazebo_joint_dynamics joint_name="${cabin_to_swing_joint_name}" stiffness="3000" damping="0.1"/>
-    <xacro:gazebo_joint_dynamics joint_name="${left_spin_to_skid_joint_name}" stiffness="3000" damping="0.1"/>
-    <xacro:gazebo_joint_dynamics joint_name="${left_free_to_skid_joint_name}" stiffness="3000" damping="0.1"/>
-    <xacro:gazebo_joint_dynamics joint_name="${right_spin_to_skid_joint_name}" stiffness="3000" damping="0.1"/>
-    <xacro:gazebo_joint_dynamics joint_name="${right_free_to_skid_joint_name}" stiffness="3000" damping="0.1"/>
+    <xacro:gazebo_joint_dynamics joint_name="${excavator_slew_joint_name}" stiffness="1000" damping="0.1"/>
+    <xacro:gazebo_joint_dynamics joint_name="${plow_to_base_joint_name}" stiffness="1000" damping="0.1"/>
+    <xacro:gazebo_joint_dynamics joint_name="${arm_to_bucket_joint_name}" stiffness="1000" damping="0.1"/>
+    <xacro:gazebo_joint_dynamics joint_name="${boom_to_arm_joint_name}" stiffness="1000" damping="0.1"/>
+    <xacro:gazebo_joint_dynamics joint_name="${swing_to_boom_joint_name}" stiffness="1000" damping="0.1"/>
+    <xacro:gazebo_joint_dynamics joint_name="${cabin_to_swing_joint_name}" stiffness="1000" damping="0.1"/>
+    <xacro:gazebo_joint_dynamics joint_name="${left_spin_to_skid_joint_name}" stiffness="1000" damping="0.1"/>
+    <xacro:gazebo_joint_dynamics joint_name="${left_free_to_skid_joint_name}" stiffness="1000" damping="0.1"/>
+    <xacro:gazebo_joint_dynamics joint_name="${right_spin_to_skid_joint_name}" stiffness="1000" damping="0.1"/>
+    <xacro:gazebo_joint_dynamics joint_name="${right_free_to_skid_joint_name}" stiffness="1000" damping="0.1"/>
     <xacro:simple_transmission name="${excavator_slew_joint_name}"/>
     <xacro:simple_transmission name="${plow_to_base_joint_name}"/>
@@ -70,9 +81,9 @@
             </hardware>
             <xacro:gazebo_ros2_control_joints_effort name="${excavator_slew_joint_name}" effort_lim="100000"/>
-            <xacro:gazebo_ros2_control_joints_effort name="${plow_to_base_joint_name}"  effort_lim="100000"/>
+            <xacro:gazebo_ros2_control_joints_effort name="${cabin_to_swing_joint_name}"  effort_lim="100000"/>
+            <xacro:gazebo_ros2_control_joints_effort name="${swing_to_boom_joint_name}"  effort_lim="100000"/>
             <xacro:gazebo_ros2_control_joints_effort name="${arm_to_bucket_joint_name}"  effort_lim="100000"/>
             <xacro:gazebo_ros2_control_joints_effort name="${boom_to_arm_joint_name}"  effort_lim="100000"/>
-            <xacro:gazebo_ros2_control_joints_effort name="${swing_to_boom_joint_name}"  effort_lim="100000"/>
-            <xacro:gazebo_ros2_control_joints_effort name="${cabin_to_swing_joint_name}"  effort_lim="100000"/>
+            <xacro:gazebo_ros2_control_joints_effort name="${plow_to_base_joint_name}"  effort_lim="100000"/>
             <!-- <xacro:gazebo_ros2_control_joints_velocity name="${excavator_slew_joint_name}" velocity_lim="1.0"/>
             <xacro:gazebo_ros2_control_joints_velocity name="${plow_to_base_joint_name}"  velocity_lim="1.0"/>
@@ -81,4 +92,10 @@
             <xacro:gazebo_ros2_control_joints_velocity name="${swing_to_boom_joint_name}"  velocity_lim="1.0"/>
             <xacro:gazebo_ros2_control_joints_velocity name="${cabin_to_swing_joint_name}"  velocity_lim="1.0"/> -->
+            <xacro:gazebo_ros2_control_joints_position name="${excavator_slew_joint_name}" position_lim="1"/>
+            <xacro:gazebo_ros2_control_joints_position name="${cabin_to_swing_joint_name}"  position_lim="1"/>
+            <xacro:gazebo_ros2_control_joints_position name="${swing_to_boom_joint_name}"  position_lim="1"/>
+            <xacro:gazebo_ros2_control_joints_position name="${arm_to_bucket_joint_name}"  position_lim="1"/>
+            <xacro:gazebo_ros2_control_joints_position name="${boom_to_arm_joint_name}"  position_lim="1"/>
+            <xacro:gazebo_ros2_control_joints_position name="${plow_to_base_joint_name}"  position_lim="1"/>
         </ros2_control>
         <gazebo>

File: sambot_description/urdf/joints.xacro (robot description, xacro)
@@ -108,5 +108,5 @@
         <child link="${boom_link_name}" />
         <axis xyz="0 0 1"/>
-        <limit effort="20000" velocity="5" lower="-1" upper="1" />
+        <limit effort="20000" velocity="5" lower="-0.4" upper="1" />
         <!-- <xacro:dynamics dyn_damping="0.1" dyn_friction="0.2"/> -->
     </joint>

File: sambot_description/urdf/robot.urdf (robot description, URDF)
Before this commit: robot excavator, 16 links, 15 joints
Joints:
- joint arm_to_bucket: limit lower=-1.2217304763960306069 upper=0.87266462599716476678 effort=10000 velocity=5 -> lower=-1.2217304763960306069 upper=0.87266462599716476678 effort=20000 velocity=5
- joint boom_to_arm: limit lower=-0.5 upper=1.57 effort=10000 velocity=5 -> lower=-0.5 upper=1.57 effort=20000 velocity=5
- joint cabin_to_swing: limit lower=-1 upper=1.57 effort=10000 velocity=5 -> lower=-0.1 upper=0.1 effort=20000 velocity=5; origin xyz=-0.040707723917193447405 -0.80673603465099630316 0.38039999999999996039 rpy=3.141592653589793116 4.8797124238540929311e-17 0.21446312817660284633 -> xyz=-0.040707723917193447405 -0.80673603465099630316 0.38039999999999996039 rpy=3.141592653589793116 4.8797124238540929311e-17 0
- joint excavator_slew: limit effort=10000 velocity=5 -> effort=20000 velocity=5
- joint left_front_to_turret: limit effort=10000 velocity=5 -> effort=20000 velocity=5
- joint left_spinning_to_turret: limit effort=10000 velocity=5 -> effort=20000 velocity=5
- joint plow_to_base: limit lower=0.2 upper=0 effort=10000 velocity=5 -> lower=0.2 upper=0 effort=20000 velocity=5
- joint right_front_to_turret: limit effort=10000 velocity=5 -> effort=20000 velocity=5
- joint right_spinning_to_turret: limit effort=10000 velocity=5 -> effort=20000 velocity=5
- joint swing_to_boom: limit lower=-0.4 upper=0.4 effort=10000 velocity=5 -> lower=-1 upper=1 effort=20000 velocity=5
