Commit message: pre position control changes

File: sambot_description/urdf/dynamics.xacro (robot description, xacro)
@@ -16,4 +16,5 @@
     <xacro:macro name="gazebo_ros2_control_joints_effort" params="name effort_lim">
         <joint name="${name}">
+            <hardwareInterface>hardware_interface/EffortJointInterface</hardwareInterface>
             <command_interface name="effort">
                 <param name="min">${-effort_lim}</param>
@@ -51,8 +52,8 @@
             <type>transmission_interface/SimpleTransmission</type>
             <joint name="${name}">
-            <hardwareInterface>effort</hardwareInterface>
+            <hardwareInterface>hardware_interface/EffortJointInterface</hardwareInterface>
             </joint>
             <actuator name="${name}_motor">
-            <hardwareInterface>effort</hardwareInterface>
+            <hardwareInterface>hardware_interface/EffortJointInterface</hardwareInterface>
             <mechanicalReduction>1</mechanicalReduction>
             </actuator>
@@ -80,10 +81,10 @@
                 <plugin>gazebo_ros2_control/GazeboSystem</plugin>
             </hardware>
-            <xacro:gazebo_ros2_control_joints_effort name="${excavator_slew_joint_name}" effort_lim="100000"/>
-            <xacro:gazebo_ros2_control_joints_effort name="${cabin_to_swing_joint_name}"  effort_lim="100000"/>
-            <xacro:gazebo_ros2_control_joints_effort name="${swing_to_boom_joint_name}"  effort_lim="100000"/>
-            <xacro:gazebo_ros2_control_joints_effort name="${arm_to_bucket_joint_name}"  effort_lim="100000"/>
-            <xacro:gazebo_ros2_control_joints_effort name="${boom_to_arm_joint_name}"  effort_lim="100000"/>
-            <xacro:gazebo_ros2_control_joints_effort name="${plow_to_base_joint_name}"  effort_lim="100000"/>
+            <xacro:gazebo_ros2_control_joints_effort name="${excavator_slew_joint_name}" effort_lim="20000"/>
+            <xacro:gazebo_ros2_control_joints_effort name="${cabin_to_swing_joint_name}"  effort_lim="20000"/>
+            <xacro:gazebo_ros2_control_joints_effort name="${swing_to_boom_joint_name}"  effort_lim="20000"/>
+            <xacro:gazebo_ros2_control_joints_effort name="${arm_to_bucket_joint_name}"  effort_lim="20000"/>
+            <xacro:gazebo_ros2_control_joints_effort name="${boom_to_arm_joint_name}"  effort_lim="20000"/>
+            <xacro:gazebo_ros2_control_joints_effort name="${plow_to_base_joint_name}"  effort_lim="20000"/>
             <!-- <xacro:gazebo_ros2_control_joints_velocity name="${excavator_slew_joint_name}" velocity_lim="1.0"/>
             <xacro:gazebo_ros2_control_joints_velocity name="${plow_to_base_joint_name}"  velocity_lim="1.0"/>
@@ -92,4 +93,5 @@
             <xacro:gazebo_ros2_control_joints_velocity name="${swing_to_boom_joint_name}"  velocity_lim="1.0"/>
             <xacro:gazebo_ros2_control_joints_velocity name="${cabin_to_swing_joint_name}"  velocity_lim="1.0"/> -->
+<!--
             <xacro:gazebo_ros2_control_joints_position name="${excavator_slew_joint_name}" position_lim="1"/>
             <xacro:gazebo_ros2_control_joints_position name="${cabin_to_swing_joint_name}"  position_lim="1"/>
@@ -97,8 +99,8 @@
             <xacro:gazebo_ros2_control_joints_position name="${arm_to_bucket_joint_name}"  position_lim="1"/>
             <xacro:gazebo_ros2_control_joints_position name="${boom_to_arm_joint_name}"  position_lim="1"/>
-            <xacro:gazebo_ros2_control_joints_position name="${plow_to_base_joint_name}"  position_lim="1"/>
+            <xacro:gazebo_ros2_control_joints_position name="${plow_to_base_joint_name}"  position_lim="1"/> -->
         </ros2_control>
         <gazebo>
-            <plugin filename="libgazebo_ros2_control.so" name="gazebo_ros2_control">
+            <plugin name="gazebo_ros2_control" filename="libgazebo_ros2_control.so">
                 <parameters>$(find sambot_description)/params/ros2_controllers.yaml</parameters>
             </plugin>

File: sambot_description/urdf/joints.xacro (robot description, xacro)
@@ -108,5 +108,5 @@
         <child link="${boom_link_name}" />
         <axis xyz="0 0 1"/>
-        <limit effort="20000" velocity="5" lower="-0.4" upper="1" />
+        <limit effort="20000" velocity="1.0" lower="-0.4" upper="1" />
         <!-- <xacro:dynamics dyn_damping="0.1" dyn_friction="0.2"/> -->
     </joint>

Commit message: ignition control

File: sambot_description/urdf/dynamics.xacro (robot description, xacro)
@@ -7,40 +7,16 @@
             <damping>${damping}</damping>
             <pid>
-                <p>100</p>
+                <p>1</p>
                 <i>0</i>
-                <d>0.1</d>
+                <d>0</d>
             </pid>
-            <!-- <dynamics damping="0.1" friction="0.2"/> -->
+            <dynamics damping="5" friction="0.2"/>
         </gazebo>
-    </xacro:macro>
-    <xacro:macro name="gazebo_ros2_control_joints_effort" params="name effort_lim">
-        <joint name="${name}">
-            <hardwareInterface>hardware_interface/EffortJointInterface</hardwareInterface>
-            <command_interface name="effort">
-                <param name="min">${-effort_lim}</param>
-                <param name="max">${effort_lim}</param>
-            </command_interface>
-            <state_interface name="position"/>
-            <state_interface name="velocity"/>
-            <!-- <state_interface name="effort"/> -->
-        </joint>
     </xacro:macro>
     <xacro:macro name="gazebo_ros2_control_joints_velocity" params="name velocity_lim">
         <joint name="${name}">
-        <hardwareInterface>hardware_interface/VelocityJointInterface</hardwareInterface>
             <command_interface name="velocity">
                 <param name="min">${-velocity_lim}</param>
                 <param name="max">${velocity_lim}</param>
-            </command_interface>
-            <state_interface name="position"/>
-            <state_interface name="velocity"/>
-            <!-- <state_interface name="effort"/> -->
-        </joint>
-    </xacro:macro>
-    <xacro:macro name="gazebo_ros2_control_joints_position" params="name position_lim">
-        <joint name="${name}">
-            <command_interface name="position">
-                <param name="min">${-position_lim}</param>
-                <param name="max">${position_lim}</param>
             </command_interface>
             <state_interface name="position"/>
@@ -61,14 +37,14 @@
         </transmission>
     </xacro:macro>
-    <xacro:gazebo_joint_dynamics joint_name="${excavator_slew_joint_name}" stiffness="1000" damping="0.1"/>
-    <xacro:gazebo_joint_dynamics joint_name="${plow_to_base_joint_name}" stiffness="1000" damping="0.1"/>
-    <xacro:gazebo_joint_dynamics joint_name="${arm_to_bucket_joint_name}" stiffness="10000" damping="500"/>
-    <xacro:gazebo_joint_dynamics joint_name="${boom_to_arm_joint_name}" stiffness="1000" damping="0.1"/>
-    <xacro:gazebo_joint_dynamics joint_name="${swing_to_boom_joint_name}" stiffness="1000" damping="0.1"/>
-    <xacro:gazebo_joint_dynamics joint_name="${cabin_to_swing_joint_name}" stiffness="1000" damping="0.1"/>
-    <xacro:gazebo_joint_dynamics joint_name="${left_spin_to_skid_joint_name}" stiffness="1000" damping="0.1"/>
-    <xacro:gazebo_joint_dynamics joint_name="${left_free_to_skid_joint_name}" stiffness="1000" damping="0.1"/>
-    <xacro:gazebo_joint_dynamics joint_name="${right_spin_to_skid_joint_name}" stiffness="1000" damping="0.1"/>
-    <xacro:gazebo_joint_dynamics joint_name="${right_free_to_skid_joint_name}" stiffness="1000" damping="0.1"/>
+    <!-- <xacro:gazebo_joint_dynamics joint_name="${excavator_slew_joint_name}" stiffness="100" damping="5"/>
+    <xacro:gazebo_joint_dynamics joint_name="${plow_to_base_joint_name}" stiffness="100" damping="5"/>
+    <xacro:gazebo_joint_dynamics joint_name="${arm_to_bucket_joint_name}" stiffness="100" damping="5"/>
+    <xacro:gazebo_joint_dynamics joint_name="${boom_to_arm_joint_name}" stiffness="100" damping="5"/>
+    <xacro:gazebo_joint_dynamics joint_name="${swing_to_boom_joint_name}" stiffness="100" damping="5"/>
+    <xacro:gazebo_joint_dynamics joint_name="${cabin_to_swing_joint_name}" stiffness="100" damping="5"/>
+    <xacro:gazebo_joint_dynamics joint_name="${left_spin_to_skid_joint_name}" stiffness="100" damping="5"/>
+    <xacro:gazebo_joint_dynamics joint_name="${left_free_to_skid_joint_name}" stiffness="100" damping="5"/>
+    <xacro:gazebo_joint_dynamics joint_name="${right_spin_to_skid_joint_name}" stiffness="100" damping="5"/>
+    <xacro:gazebo_joint_dynamics joint_name="${right_free_to_skid_joint_name}" stiffness="100" damping="5"/> -->
     <xacro:simple_transmission name="${excavator_slew_joint_name}"/>
     <xacro:simple_transmission name="${plow_to_base_joint_name}"/>
@@ -79,13 +55,10 @@
     <xacro:macro name="dynamics_plugins">
         <ros2_control name="GazeboSystem" type="system">
+            <!-- <hardware>
+                <plugin>gazebo_ros2_control/GazeboSystem</plugin>
+            </hardware> -->
             <hardware>
-                <plugin>gazebo_ros2_control/GazeboSystem</plugin>
+                <plugin>gz_ros2_control/GazeboSimSystem</plugin>
             </hardware>
-            <xacro:gazebo_ros2_control_joints_effort name="${excavator_slew_joint_name}" effort_lim="20000"/>
-            <xacro:gazebo_ros2_control_joints_effort name="${cabin_to_swing_joint_name}"  effort_lim="20000"/>
-            <xacro:gazebo_ros2_control_joints_effort name="${swing_to_boom_joint_name}"  effort_lim="20000"/>
-            <xacro:gazebo_ros2_control_joints_effort name="${arm_to_bucket_joint_name}"  effort_lim="20000"/>
-            <xacro:gazebo_ros2_control_joints_effort name="${boom_to_arm_joint_name}"  effort_lim="20000"/>
-            <xacro:gazebo_ros2_control_joints_effort name="${plow_to_base_joint_name}"  effort_lim="20000"/>
             <xacro:gazebo_ros2_control_joints_velocity name="${excavator_slew_joint_name}" velocity_lim="1.0"/>
             <xacro:gazebo_ros2_control_joints_velocity name="${plow_to_base_joint_name}"  velocity_lim="1.0"/>
@@ -94,17 +67,13 @@
             <xacro:gazebo_ros2_control_joints_velocity name="${swing_to_boom_joint_name}"  velocity_lim="1.0"/>
             <xacro:gazebo_ros2_control_joints_velocity name="${cabin_to_swing_joint_name}"  velocity_lim="1.0"/>
-            <xacro:gazebo_ros2_control_joints_position name="${excavator_slew_joint_name}" position_lim="${pi}"/>
-            <xacro:gazebo_ros2_control_joints_position name="${cabin_to_swing_joint_name}"  position_lim="${pi}"/>
-            <xacro:gazebo_ros2_control_joints_position name="${swing_to_boom_joint_name}"  position_lim="${pi}"/>
-            <xacro:gazebo_ros2_control_joints_position name="${arm_to_bucket_joint_name}"  position_lim="${pi}"/>
-            <xacro:gazebo_ros2_control_joints_position name="${boom_to_arm_joint_name}"  position_lim="${pi}"/>
-            <xacro:gazebo_ros2_control_joints_position name="${plow_to_base_joint_name}"  position_lim="${pi}"/>
         </ros2_control>
         <gazebo>
-            <plugin name="gazebo_ros2_control" filename="libgazebo_ros2_control.so">
-                <parameters>$(find sambot_description)/params/ros2_controllers.yaml</parameters>
+            <!-- <plugin name="gazebo_ros2_control" filename="libgazebo_ros2_control.so"> -->
+            <plugin filename="gz_ros2_control-system" name="gz_ros2_control::GazeboSimROS2ControlPlugin">
+                <parameters>$(find sambot_description)/params/vc.yaml</parameters>
+                <controller_manager_name>controller_manager</controller_manager_name>
             </plugin>
         </gazebo>
-        <gazebo>
+        <!-- <gazebo>
             <plugin name="two_wheeled_robot_diff_drive" filename="libgazebo_ros_diff_drive.so">
                 <num_wheel_pairs>2</num_wheel_pairs>
@@ -125,5 +94,5 @@
                 <robot_base_frame>base_link</robot_base_frame>
             </plugin>
-        </gazebo>
+        </gazebo> -->
     </xacro:macro>
 </robot>

File: sambot_description/urdf/params.xacro (robot description, xacro)
@@ -45,5 +45,4 @@
     <xacro:property name="cabin_base_material" value="0.2314 0.3804 0.7059 1.0"/>
     <xacro:property name="cabin_base_inertial" value="3175.1655302028038932 -269.97312494382822479 167.61780128589879268 2627.6328649732372469 -193.85494965010886403 3742.616047274826542"/>
-    <!-- TURRET PARAMS -->
     <xacro:property name="turret_base_mesh" value="${mesh_root}/compact_excavator_frame_body.stl"/>
     <xacro:property name="turret_base_origin" value="0 0 0"/>
@@ -54,5 +53,4 @@
     <xacro:property name="turret_base_material" value="0.9176 0.9176 0.9176 1.0"/>
     <xacro:property name="turret_base_inertial" value="103.54309263053609413 2.8689912175751035583 -0.26918599165092144121 71.550382439979060223 -8.7881744003938315757 164.71779214088334697"/>
-    <!-- LEFT SPINNING (BACK) WHEEL -->
     <xacro:property name="left_spinning_wheel_link_mesh" value="${mesh_root}/compact_excavator_main_drive_wheel.stl"/>
     <xacro:property name="left_spinning_wheel_link_origin" value="0 -2.0816681711721685133e-17 -0.015000000000000124345"/>
@@ -63,5 +61,4 @@
     <xacro:property name="left_spinning_wheel_link_mass" value="35.986291345795820007"/>
     <xacro:property name="left_spinning_wheel_link_inertial" value="0.20071737580058110484 2.1151248144254331483e-17 7.9696042408110000254e-05 0.20066206838835709547 2.9623558171777900037e-16 0.29333573070696433716"/>
-    <!-- RIGHT SPINNING (BACK) WHEEL -->
     <xacro:property name="right_spinning_wheel_link_mesh" value="${mesh_root}/compact_excavator_main_drive_wheel.stl"/>
     <xacro:property name="right_spinning_wheel_link_origin" value="-6.9388939039072283776e-18 0 -0.015000000000000013323"/>
@@ -72,5 +69,4 @@
     <xacro:property name="right_spinning_wheel_link_mass" value="35.986291345795820007"/>
     <xacro:property name="right_spinning_wheel_link_inertial" value="0.20071737580058127137 6.1250580134766935832e-18 7.9696042408110027359e-05 0.20066206838835703996 2.9623106429686494369e-16 0.29333573070696433716"/>
-    <!-- LEFT FRONT WHEEL -->
     <xacro:property name="left_front_wheel_link_mesh" value="${mesh_root}/compact_excavator_front_wheel.stl"/>
     <xacro:property name="left_front_wheel_link_origin" value="1.1102230246251565404e-16 -1.1102230246251565404e-16 -0.032500000000000084377"/>
@@ -81,5 +77,4 @@
     <xacro:property name="left_front_wheel_link_mass" value="17.64673591392957519"/>
     <xacro:property name="left_front_wheel_link_inertial" value="0.153078316536178205 1.0629206596102168903e-17 2.6922495826861160064e-17 0.15307831653617814949 6.9747558075870228735e-33 0.29963755764746907717"/>
-    <!-- RIGHT FRONT WHEEL -->
     <xacro:property name="right_front_wheel_link_mesh" value="${mesh_root}/compact_excavator_front_wheel.stl"/>
     <xacro:property name="right_front_wheel_link_origin" value="-2.7755575615628913511e-17 0 -0.032500000000000084377"/>
@@ -90,5 +85,4 @@
     <xacro:property name="right_front_wheel_link_mass" value="17.64673591392957519"/>
     <xacro:property name="right_front_wheel_link_inertial" value="0.153078316536178205 -1.0629206596102168903e-17 2.6922495826861160064e-17 0.15307831653617814949 6.9747558075870228735e-33 0.29963755764746907717"/>
-    <!-- PLOW -->
     <xacro:property name="push_blade_base_mesh" value="${mesh_root}/push_blade_bucket.stl"/>
     <xacro:property name="push_blade_base_origin" value="-0.021564399534920564161 1.0799900599760599018 -0.25500000000000000444"/>
@@ -99,5 +93,4 @@
     <xacro:property name="push_blade_base_mass" value="147.01808168083425699"/>
     <xacro:property name="push_blade_base_inertial" value="31.881096131626421197 0.91247385061899932701 -1.6212090668492922982e-05 21.196220352263214437 4.9900082202379639952e-06 13.169227707961496776"/>
-    <!-- SWING -->
     <xacro:property name="swing_base_mesh" value="${mesh_root}/part01_pin_1.stl"/>
     <xacro:property name="swing_base_origin" value="2.7755575615628913511e-17 0.074999999999999955591 -0.14999999999999996669"/>
@@ -108,5 +101,4 @@
     <xacro:property name="swing_base_mass" value="98.140190062279060612"/>
     <xacro:property name="swing_base_inertial" value="2.6085778666185075458 0.040227300901953748358 0.42136783119553594679 3.1665232143977135593 -0.15916376835413623136 1.7889951810686841593"/>
-    <!-- BOOM -->
     <xacro:property name="boom_base_mesh" value="${mesh_root}/part02.stl"/>
     <xacro:property name="boom_base_origin" value="0 -1.1102230246251565404e-16 -0.079999999999999987788"/>
@@ -117,5 +109,4 @@
     <xacro:property name="boom_base_mass" value="694.17793513858055121"/>
     <xacro:property name="boom_base_inertial" value="242.81245205849677404 71.370938403077758494 0.0065905643878567711502 49.641340591529456105 -0.034260052091464154866 289.83702909122945357"/>
-    <!-- ARM -->
     <xacro:property name="arm_base_mesh" value="${mesh_root}/part03.stl"/>
     <xacro:property name="arm_base_origin" value="0 -2.2204460492503130808e-16 -0.054999999999999882316"/>
@@ -126,5 +117,4 @@
     <xacro:property name="arm_base_mass" value="265.34907807560875881"/>
     <xacro:property name="arm_base_inertial" value="57.599134249663784146 0.078442580554215754485 0.0049826290162324230956 1.8968981412117758012 0.02459901605653430981 58.868680211308259231"/>
-    <!-- BUCKET(S) -->
     <xacro:property name="bucket_mesh1" value="${mesh_root}/part04.stl"/>
     <xacro:property name="bucket_mesh1_origin" value="0.060000000000000053291 0.14000000000000012434 0.054999999999999993339"/>
@@ -143,10 +133,8 @@
     <xacro:property name="bucket_base_mass" value="132.70765933863819441"/>
     <xacro:property name="bucket_base_inertial" value="14.03567187790122972 -1.6652440163767181502 0.0020270508814650067472 6.8549730106956987541 0.0040437120644442776929 11.610921270718170817"/>
-    <!-- SKID WHEELS FOR DIFF DRIVE -->
     <xacro:property name="rubber_density" value="1100"/>
     <xacro:property name="wheel_radius" value="0.25"/>
     <xacro:property name="wheel_length" value="0.2"/>
     <xacro:macro name="skid_wheel" params="wheel_name mu1 mu2">
-        <!-- MULTIPLIED BY 100 TO ANCHOR -->
         <xacro:property name="wheel_mass" value="${100*3.1415*(wheel_radius**2)*wheel_length*rubber_density}"/>
         <xacro:property name="wheel_ixx" value="${(1/12)*wheel_mass*(3*wheel_radius**2 + wheel_length**2)}"/>
