Commit message: testing non functional turning

File: earth_gz_ign/urdf/robot.xacro (robot description, xacro)
@@ -4,5 +4,12 @@
     <xacro:include filename="$(find earth_gz_ign)/urdf/joints.xacro" />
     <xacro:include filename="$(find earth_gz_ign)/urdf/dynamics.xacro" />
+    <link name="world"/>
     <link name="base_link"/>
+    <joint name="temp_joint" type="fixed">
+        <origin xyz="0 0 3" rpy="0 1.57 0"/>
+        <parent link="world"/>
+        <child link="base_link"/>
+        <axis xyz="0 0 1"/>
+    </joint>
     <link name="cabin_base">
         <visual>
