Commit message: updated name to earth_gz_ign

File: earth_gz_ign/urdf/dynamics.xacro (robot description, xacro)
@@ -1,5 +1,5 @@
 <?xml version="1.0"?>
 <robot xmlns:xacro="http://ros.org/wiki/xacro">
-    <xacro:include filename="$(find sambot_description)/urdf/params.xacro"/>
+    <xacro:include filename="$(find earth_gz_ign)/urdf/params.xacro"/>
     <xacro:macro name="gazebo_joint_dynamics" params="joint_name stiffness damping">
         <gazebo reference="${joint_name}">
@@ -71,5 +71,5 @@
             <!-- <plugin name="gazebo_ros2_control" filename="libgazebo_ros2_control.so"> -->
             <plugin filename="gz_ros2_control-system" name="gz_ros2_control::GazeboSimROS2ControlPlugin">
-                <parameters>$(find sambot_description)/params/vc.yaml</parameters>
+                <parameters>$(find earth_gz_ign)/params/vc.yaml</parameters>
                 <controller_manager_name>controller_manager</controller_manager_name>
             </plugin>

File: earth_gz_ign/urdf/dynamics_effort.xacro (robot description, xacro)
@@ -1,5 +1,5 @@
 <?xml version="1.0"?>
 <robot xmlns:xacro="http://ros.org/wiki/xacro">
-    <xacro:include filename="$(find sambot_description)/urdf/params.xacro"/>
+    <xacro:include filename="$(find earth_gz_ign)/urdf/params.xacro"/>
     <xacro:macro name="gazebo_joint_dynamics" params="joint_name stiffness damping">
         <gazebo reference="${joint_name}">
@@ -71,5 +71,5 @@
             <!-- <plugin name="gazebo_ros2_control" filename="libgazebo_ros2_control.so"> -->
             <plugin filename="gz_ros2_control-system" name="gz_ros2_control::GazeboSimROS2ControlPlugin">
-                <parameters>$(find sambot_description)/params/ec.yaml</parameters>
+                <parameters>$(find earth_gz_ign)/params/ec.yaml</parameters>
                 <controller_manager_name>controller_manager</controller_manager_name>
             </plugin>

File: earth_gz_ign/urdf/dynamics_effort_traj.xacro (robot description, xacro)
@@ -1,5 +1,5 @@
 <?xml version="1.0"?>
 <robot xmlns:xacro="http://ros.org/wiki/xacro">
-    <xacro:include filename="$(find sambot_description)/urdf/params.xacro"/>
+    <xacro:include filename="$(find earth_gz_ign)/urdf/params.xacro"/>
     <xacro:macro name="gazebo_joint_dynamics" params="joint_name stiffness damping">
         <gazebo reference="${joint_name}">
@@ -71,5 +71,5 @@
             <!-- <plugin name="gazebo_ros2_control" filename="libgazebo_ros2_control.so"> -->
             <plugin filename="gz_ros2_control-system" name="gz_ros2_control::GazeboSimROS2ControlPlugin">
-                <parameters>$(find sambot_description)/params/etc.yaml</parameters>
+                <parameters>$(find earth_gz_ign)/params/etc.yaml</parameters>
                 <controller_manager_name>controller_manager</controller_manager_name>
             </plugin>

File: earth_gz_ign/urdf/joints.xacro (robot description, xacro)
@@ -1,5 +1,5 @@
 <?xml version="1.0"?>
 <robot xmlns:xacro="http://ros.org/wiki/xacro">
-    <xacro:include filename="$(find sambot_description)/urdf/params.xacro"/>
+    <xacro:include filename="$(find earth_gz_ign)/urdf/params.xacro"/>
     <xacro:macro name="dynamics" params="dyn_damping dyn_friction">
             <dynamics damping="${dyn_damping}" friction="${dyn_friction}"/>

File: earth_gz_ign/urdf/params.xacro (robot description, xacro)
@@ -1,5 +1,5 @@
 <?xml version="1.0"?>
 <robot xmlns:xacro="http://ros.org/wiki/xacro">
-    <xacro:property name="mesh_root" value="file://$(find sambot_description)/meshes"/>
+    <xacro:property name="mesh_root" value="file://$(find earth_gz_ign)/meshes"/>
     <!-- MAIN LINK NAMES -->
     <xacro:property name="base_link_name" value="base_link"/>

File: earth_gz_ign/urdf/robot.urdf (robot description, URDF)
Before this commit: robot excavator, 16 links, 15 joints
Links:
- link arm_base: geometry collision mesh filename=file:///home/moog-2/nav2_ws/install/earth_gz_ign/share/eart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; visual mesh filename=file:///home/moog-2/nav2_ws/install/earth_gz_ign/share/eart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
- link boom_base: geometry collision mesh filename=file:///home/moog-2/nav2_ws/install/earth_gz_ign/share/eart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; visual mesh filename=file:///home/moog-2/nav2_ws/install/earth_gz_ign/share/eart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
- link bucket_base: geometry collision mesh filename=file:///home/moog-2/nav2_ws/install/earth_gz_ign/share/eart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; collision mesh filename=file:///home/moog-2/nav2_ws/install/earth_gz_ign/share/eart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
- link cabin_base: geometry collision mesh filename=file:///home/moog-2/nav2_ws/install/earth_gz_ign/share/eart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; visual mesh filename=file:///home/moog-2/nav2_ws/install/earth_gz_ign/share/eart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
- link left_front_wheel_link: geometry collision mesh filename=file:///home/moog-2/nav2_ws/install/earth_gz_ign/share/eart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; visual mesh filename=file:///home/moog-2/nav2_ws/install/earth_gz_ign/share/eart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
- link left_spinning_wheel_link: geometry collision mesh filename=file:///home/moog-2/nav2_ws/install/earth_gz_ign/share/eart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; visual mesh filename=file:///home/moog-2/nav2_ws/install/earth_gz_ign/share/eart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
- link push_blade_base: geometry collision mesh filename=file:///home/moog-2/nav2_ws/install/earth_gz_ign/share/eart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; visual mesh filename=file:///home/moog-2/nav2_ws/install/earth_gz_ign/share/eart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
- link right_front_wheel_link: geometry collision mesh filename=file:///home/moog-2/nav2_ws/install/earth_gz_ign/share/eart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; visual mesh filename=file:///home/moog-2/nav2_ws/install/earth_gz_ign/share/eart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
- link right_spinning_wheel_link: geometry collision mesh filename=file:///home/moog-2/nav2_ws/install/earth_gz_ign/share/eart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; visual mesh filename=file:///home/moog-2/nav2_ws/install/earth_gz_ign/share/eart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
- link swing_base: geometry collision mesh filename=file:///home/moog-2/nav2_ws/install/earth_gz_ign/share/eart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; visual mesh filename=file:///home/moog-2/nav2_ws/install/earth_gz_ign/share/eart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
- link turret_base: geometry collision mesh filename=file:///home/moog-2/nav2_ws/install/earth_gz_ign/share/eart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; visual mesh filename=file:///home/moog-2/nav2_ws/install/earth_gz_ign/share/eart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

File: earth_gz_ign/urdf/robot.xacro (robot description, xacro)
@@ -1,7 +1,7 @@
 <?xml version="1.0"?>
 <robot xmlns:xacro="http://www.ros.org/wiki/xacro" name="excavator">
-    <xacro:include filename="$(find sambot_description)/urdf/params.xacro" />
-    <xacro:include filename="$(find sambot_description)/urdf/joints.xacro" />
-    <xacro:include filename="$(find sambot_description)/urdf/dynamics_effort_traj.xacro" />
+    <xacro:include filename="$(find earth_gz_ign)/urdf/params.xacro" />
+    <xacro:include filename="$(find earth_gz_ign)/urdf/joints.xacro" />
+    <xacro:include filename="$(find earth_gz_ign)/urdf/dynamics.xacro" />
     <link name="base_link"/>
     <link name="cabin_base">

File: earth_gz_ign/urdf/robot_effort.xacro (robot description, xacro)
@@ -1,7 +1,7 @@
 <?xml version="1.0"?>
 <robot xmlns:xacro="http://www.ros.org/wiki/xacro" name="excavator">
-    <xacro:include filename="$(find sambot_description)/urdf/params.xacro" />
-    <xacro:include filename="$(find sambot_description)/urdf/joints.xacro" />
-    <xacro:include filename="$(find sambot_description)/urdf/dynamics.xacro" />
+    <xacro:include filename="$(find earth_gz_ign)/urdf/params.xacro" />
+    <xacro:include filename="$(find earth_gz_ign)/urdf/joints.xacro" />
+    <xacro:include filename="$(find earth_gz_ign)/urdf/dynamics_effort.xacro" />
     <link name="base_link"/>
     <link name="cabin_base">

File: earth_gz_ign/urdf/robot_effort_traj.xacro (robot description, xacro)
@@ -1,7 +1,7 @@
 <?xml version="1.0"?>
 <robot xmlns:xacro="http://www.ros.org/wiki/xacro" name="excavator">
-    <xacro:include filename="$(find sambot_description)/urdf/params.xacro" />
-    <xacro:include filename="$(find sambot_description)/urdf/joints.xacro" />
-    <xacro:include filename="$(find sambot_description)/urdf/dynamics_effort.xacro" />
+    <xacro:include filename="$(find earth_gz_ign)/urdf/params.xacro" />
+    <xacro:include filename="$(find earth_gz_ign)/urdf/joints.xacro" />
+    <xacro:include filename="$(find earth_gz_ign)/urdf/dynamics_effort_traj.xacro" />
     <link name="base_link"/>
     <link name="cabin_base">

Commit message: added cmd_vel movement

File: earth_gz_ign/urdf/dynamics.xacro (robot description, xacro)
@@ -74,13 +74,15 @@
                 <controller_manager_name>controller_manager</controller_manager_name>
             </plugin>
-            <plugin
-                filename="libignition-gazebo-diff-drive-system.so"
-                name="ignition::gazebo::systems::DiffDrive">
-                <left_joint>left_spinning_to_turret</left_joint>
-                <right_joint>right_spinning_to_turret</right_joint>
-                <wheel_separation>1.2</wheel_separation>
-                <wheel_radius>0.4</wheel_radius>
-                <odom_publish_frequency>1</odom_publish_frequency>
-                <topic>cmd_vel</topic>
+            <plugin filename="gz-sim-diff-drive-system" name="gz::sim::systems::DiffDrive">
+            <left_joint>left_spinning_to_turret</left_joint>
+            <right_joint>right_spinning_to_turret</right_joint>
+            <wheel_separation>1.2</wheel_separation>
+            <wheel_radius>${wheel_radius}</wheel_radius>
+            <max_linear_acceleration>0.1</max_linear_acceleration>
+            <topic>/demo/cmd_vel</topic>
+            <odom_topic>/demo/odom</odom_topic>
+            <tf_topic>/tf</tf_topic>
+            <frame_id>odom</frame_id>
+            <child_frame_id>base_link</child_frame_id>
             </plugin>
         </gazebo>

File: earth_gz_ign/urdf/robot.urdf (robot description, URDF)
Before this commit: robot excavator, 16 links, 15 joints
Links:
- link arm_base: geometry collision mesh filename=file:///home/moog-2/christo/ros2_ws/install/earth_gz_ign/sh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; visual mesh filename=file:///home/moog-2/christo/ros2_ws/install/earth_gz_ign/sh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
- link boom_base: geometry collision mesh filename=file:///home/moog-2/christo/ros2_ws/install/earth_gz_ign/sh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; visual mesh filename=file:///home/moog-2/christo/ros2_ws/install/earth_gz_ign/sh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
- link bucket_base: geometry collision mesh filename=file:///home/moog-2/christo/ros2_ws/install/earth_gz_ign/sh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; collision mesh filename=file:///home/moog-2/christo/ros2_ws/install/earth_gz_ign/sh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
- link cabin_base: geometry collision mesh filename=file:///home/moog-2/christo/ros2_ws/install/earth_gz_ign/sh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; visual mesh filename=file:///home/moog-2/christo/ros2_ws/install/earth_gz_ign/sh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
- link left_front_wheel_link: geometry collision mesh filename=file:///home/moog-2/christo/ros2_ws/install/earth_gz_ign/sh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; visual mesh filename=file:///home/moog-2/christo/ros2_ws/install/earth_gz_ign/sh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
- link left_spinning_wheel_link: geometry collision mesh filename=file:///home/moog-2/christo/ros2_ws/install/earth_gz_ign/sh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; visual mesh filename=file:///home/moog-2/christo/ros2_ws/install/earth_gz_ign/sh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
- link push_blade_base: geometry collision mesh filename=file:///home/moog-2/christo/ros2_ws/install/earth_gz_ign/sh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; visual mesh filename=file:///home/moog-2/christo/ros2_ws/install/earth_gz_ign/sh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
- link right_front_wheel_link: geometry collision mesh filename=file:///home/moog-2/christo/ros2_ws/install/earth_gz_ign/sh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; visual mesh filename=file:///home/moog-2/christo/ros2_ws/install/earth_gz_ign/sh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
- link right_spinning_wheel_link: geometry collision mesh filename=file:///home/moog-2/christo/ros2_ws/install/earth_gz_ign/sh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; visual mesh filename=file:///home/moog-2/christo/ros2_ws/install/earth_gz_ign/sh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
- link swing_base: geometry collision mesh filename=file:///home/moog-2/christo/ros2_ws/install/earth_gz_ign/sh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; visual mesh filename=file:///home/moog-2/christo/ros2_ws/install/earth_gz_ign/sh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
- link turret_base: geometry collision mesh filename=file:///home/moog-2/christo/ros2_ws/install/earth_gz_ign/sh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; visual mesh filename=file:///home/moog-2/christo/ros2_ws/install/earth_gz_ign/sh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

Commit message: fixed bridge issues

File: earth_gz_ign/urdf/dynamics.xacro (robot description, xacro)
@@ -79,5 +79,5 @@
             <wheel_separation>1.2</wheel_separation>
             <wheel_radius>${wheel_radius}</wheel_radius>
-            <max_linear_acceleration>0.1</max_linear_acceleration>
+            <max_linear_acceleration>0.5</max_linear_acceleration>
             <topic>/demo/cmd_vel</topic>
             <odom_topic>/demo/odom</odom_topic>
@@ -85,4 +85,10 @@
             <frame_id>odom</frame_id>
             <child_frame_id>base_link</child_frame_id>
+            </plugin>
+            <plugin
+                filename="gz-sim-pose-publisher-system"
+                name="gz::sim::systems::PosePublisher">
+                <use_pose_vector_msg>true</use_pose_vector_msg>
+                <publish_nested_model_pose>true</publish_nested_model_pose>
             </plugin>
         </gazebo>

File: earth_gz_ign/urdf/params.xacro (robot description, xacro)
@@ -137,5 +137,5 @@
     <xacro:property name="wheel_length" value="0.2"/>
     <xacro:macro name="skid_wheel" params="wheel_name mu1 mu2">
-        <xacro:property name="wheel_mass" value="${100*3.1415*(wheel_radius**2)*wheel_length*rubber_density}"/>
+        <xacro:property name="wheel_mass" value="${3.1415*(wheel_radius**2)*wheel_length*rubber_density}"/>
         <xacro:property name="wheel_ixx" value="${(1/12)*wheel_mass*(3*wheel_radius**2 + wheel_length**2)}"/>
         <xacro:property name="wheel_iyy" value="${(1/12)*wheel_mass*(3*wheel_radius**2 + wheel_length**2)}"/>

Commit message: slight turning now changed slips to 1.0

File: earth_gz_ign/urdf/dynamics.xacro (robot description, xacro)
@@ -76,5 +76,7 @@
             <plugin filename="gz-sim-diff-drive-system" name="gz::sim::systems::DiffDrive">
             <left_joint>left_spinning_to_turret</left_joint>
+            <left_joint>left_front_to_turret</left_joint>
             <right_joint>right_spinning_to_turret</right_joint>
+            <right_joint>right_front_to_turret</right_joint>
             <wheel_separation>1.2</wheel_separation>
             <wheel_radius>${wheel_radius}</wheel_radius>

File: earth_gz_ign/urdf/joints.xacro (robot description, xacro)
@@ -44,6 +44,6 @@
         <child link="${left_spinning_wheel_link_name}" />
         <axis xyz="0 0 1"/>
-        <limit effort="100000" velocity="1" />
-        <xacro:dynamics dyn_damping="10000" dyn_friction="0.2"/>
+        <limit effort="100000" velocity="0.5" />
+        <!-- <xacro:dynamics dyn_damping="100000" dyn_friction="10"/>   -->
     </joint>
     <joint name="${right_spinning_to_turret_joint_name}" type="continuous">
@@ -52,6 +52,6 @@
         <child link="${right_spinning_wheel_link_name}" />
         <axis xyz="0 0 1"/>
-        <limit effort="10000" velocity="1" />
-        <xacro:dynamics dyn_damping="10000" dyn_friction="0.2"/>
+        <limit effort="10000" velocity="0.5" />
+        <!-- <xacro:dynamics dyn_damping="100000" dyn_friction="10"/>   -->
     </joint>
     <joint name="${left_front_to_turret_joint_name}" type="continuous">
@@ -60,6 +60,6 @@
         <child link="${left_front_wheel_link_name}" />
         <axis xyz="0 0 1"/>
-        <limit effort="100000" velocity="1" />
-        <xacro:dynamics dyn_damping="10000" dyn_friction="0.2"/>
+        <limit effort="100000" velocity="0.5" />
+        <!-- <xacro:dynamics dyn_damping="100000" dyn_friction="10"/>   -->
     </joint>
     <joint name="${right_front_to_turret_joint_name}" type="continuous">
@@ -68,6 +68,6 @@
         <child link="${right_front_wheel_link_name}" />
         <axis xyz="0 0 1"/>
-        <limit effort="100000" velocity="1" />
-        <xacro:dynamics dyn_damping="10000" dyn_friction="0.2"/>
+        <limit effort="100000" velocity="0.5" />
+        <!-- <xacro:dynamics dyn_damping="100000" dyn_friction="10"/>   -->
     </joint>
     <joint name="${plow_to_base_joint_name}" type="revolute">

File: earth_gz_ign/urdf/params.xacro (robot description, xacro)
@@ -137,5 +137,5 @@
     <xacro:property name="wheel_length" value="0.2"/>
     <xacro:macro name="skid_wheel" params="wheel_name mu1 mu2">
-        <xacro:property name="wheel_mass" value="${3.1415*(wheel_radius**2)*wheel_length*rubber_density}"/>
+        <xacro:property name="wheel_mass" value="${2*3.1415*(wheel_radius**2)*wheel_length*rubber_density}"/>
         <xacro:property name="wheel_ixx" value="${(1/12)*wheel_mass*(3*wheel_radius**2 + wheel_length**2)}"/>
         <xacro:property name="wheel_iyy" value="${(1/12)*wheel_mass*(3*wheel_radius**2 + wheel_length**2)}"/>
@@ -158,8 +158,15 @@
             </collision>
             <surface>
+                <contact>
+                    <ode>
+                    <contact_surface_layer>0.001</contact_surface_layer>
+                    </ode>
+                </contact>
                 <friction>
                     <ode>
                         <mu>${mu1}</mu>
                         <mu2>${mu2}</mu2>
+                        <slip1>0.0</slip1>
+                        <slip2>0.0</slip2>
                     </ode>
                 </friction>

File: earth_gz_ign/urdf/robot.xacro (robot description, xacro)
@@ -4,12 +4,12 @@
     <xacro:include filename="$(find earth_gz_ign)/urdf/joints.xacro" />
     <xacro:include filename="$(find earth_gz_ign)/urdf/dynamics.xacro" />
-    <link name="world"/>
+    <!-- <link name="world"/> -->
     <link name="base_link"/>
-    <joint name="temp_joint" type="fixed">
+    <!-- <joint name="temp_joint" type="fixed">
         <origin xyz="0 0 3" rpy="0 1.57 0"/>
         <parent link="world"/>
         <child link="base_link"/>
         <axis xyz="0 0 1"/>
-    </joint>
+    </joint> -->
     <link name="cabin_base">
         <visual>
